File: crkbd-mix/pcb/crkbd-mix.sch (KiCad schematic (older format))
At the start: 87 parts, among them J1 MJ-4PP-9, J2 OLED, J3 LED, P1 i2c-pin, P2 i2c-pin, SW1 SW_PUSH, SW10 SW_PUSH, SW11 SW_PUSH, SW12 SW_PUSH, SW13 SW_PUSH, SW14 SW_PUSH, SW15 SW_PUSH, SW16 SW_PUSH, SW17 SW_PUSH, SW18 SW_PUSH, SW19 SW_PUSH, SW2 SW_PUSH, SW20 SW_PUSH, SW21 SW_PUSH, SW3 SW_PUSH, SW4 SW_PUSH, SW5 SW_PUSH, SW6 SW_PUSH, SW7 SW_PUSH, SW8 SW_PUSH, SW9 SW_PUSH, U1 ProMicro

Commit message: Replace footprints for double hotswapable
Parts:
- removed J3: LED, kbd:StripLED_rev, symbol Conn_01x03
- removed L1, L10, L11, L12, L13, L14, L15, L16, L17, L18, L19, L2, L20, L21, L3, L4, L5, L6, L7, L8, L9: SK6812MINI, kbd:SK6812MINI_rev, symbol kbd:SK6812MINI
- removed L22, L23, L24, L25, L26, L27: SK6812MINI, kbd:SK6812MINI_underglow, symbol kbd:SK6812MINI
- D1, D10, D11, D12, D13, D14, D15, D16, D17, D18, D19, D2, D20, D21, D3, D4, D5, D6, D7, D8, D9: footprint kbd:D3_TH_SMD -> kbd:D3_SMD
- J2: symbol Conn_01x04 -> Connector_Generic:Conn_01x04
- P1, P2: symbol Conn_01x01 -> Connector_Generic:Conn_01x01
- SW1, SW10, SW11, SW12, SW13, SW14, SW15, SW16, SW17, SW18, SW19, SW2, SW20, SW3, SW4, SW5, SW6, SW7, SW8, SW9: footprint kbd:MX_ALPS_PG1350_noLed -> kbd:CherryMX_KailhLowProfile_Hotswap
- SW21: footprint kbd:MX_ALPS_PG1350_noLed_1.75u -> kbd:CherryMX_KailhLowProfile_Hotswap
Connections:
- wire segments 265 -> 76
- no-connect marks 6 -> 5
