File: corne-cherry/pcb_top/corne-cherry-top-plate.kicad_pcb (KiCad board)
At the start: 2 copper layers, 132.9 x 91.4 mm, 5 parts

Commit message: Some updates
Other:
- board text added: "Corne Keyboard PCB Designed by foostan"
- board text removed: "Corne Keyboard v2.1 PCB Designed by foostan"
Changed lines of the file:
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@@
   (gr_line (start 79.5 105.5) (end 79.51 105.5) (angle 90) (layer Eco2.User) (width 2.5))
   (gr_line (start 79.5 86.75) (end 79.51 86.75) (angle 90) (layer Eco2.User) (width 2.5))
-  (gr_text "Corne Keyboard v2.1\nPCB Designed by foostan" (at 117.55 121.45) (layer B.Mask)
+  (gr_text "Corne Keyboard\nPCB Designed by foostan" (at 118.11 121.445) (layer B.Mask)
     (effects (font (size 1 1) (thickness 0.125)) (justify left mirror))
   )
-  (gr_text "Corne Keyboard v2.1\nPCB Designed by foostan" (at 98.25 121.45) (layer F.Mask)
+  (gr_text "Corne Keyboard\nPCB Designed by foostan" (at 98.74 121.445) (layer F.Mask)
     (effects (font (size 1 1) (thickness 0.125)) (justify left))
   )
