File: corne-light/pcb/corne-light.kicad_pcb (KiCad board)
At the start: 2 copper layers, 133.8 x 157.4 mm, 190 parts, among them J1 MJ-4PP-9, J10 LED, J2 OLED, J3 LED, J4 Conn_01x01, J5 LED, J6 MJ-4PP-9, J7 OLED, J8 LED, J9 Conn_01x01, SW1 SW_PUSH, SW10 SW_PUSH, SW11 SW_PUSH, SW12 SW_PUSH, SW13 SW_PUSH, SW14 SW_PUSH, SW15 SW_PUSH, SW16 SW_PUSH, SW17 SW_PUSH, SW18 SW_PUSH, SW19 SW_PUSH, SW2 SW_PUSH, SW20 SW_PUSH, SW21 SW_PUSH, SW22 SW_PUSH, SW23 SW_PUSH, SW24 SW_PUSH, SW25 SW_PUSH, SW26 SW_PUSH, SW27 SW_PUSH, SW28 SW_PUSH, SW29 SW_PUSH, SW3 SW_PUSH, SW30 SW_PUSH, SW31 SW_PUSH, SW32 SW_PUSH, SW33 SW_PUSH, SW34 SW_PUSH, SW35 SW_PUSH, SW36 SW_PUSH, SW37 SW_PUSH, SW38 SW_PUSH, SW39 SW_PUSH, SW4 SW_PUSH, SW40 SW_PUSH, SW41 SW_PUSH, SW42 SW_PUSH, SW5 SW_PUSH, SW6 SW_PUSH, SW7 SW_PUSH, SW8 SW_PUSH, SW9 SW_PUSH, U1 ProMicro, U2 ProMicro

Commit message: Brashup righ hand
Parts:
- removed the Ref** at (96.0, 104.9)
- removed the Ref** at (106.8, 104.9)
- removed the Ref** at (108.6, 98.9)
- removed the Ref** at (108.6, 104.9)
- removed the Ref** at (91.6, 107.0)
- removed the Ref** at (92.7, 107.0)
- removed the Ref** at (99.6, 98.9)
- removed the Ref** at (114.7, 107.0)
- removed the Ref** at (115.8, 107.0)
- removed the Ref** at (103.2, 104.9)
- removed the Ref** at (92.7, 93.6)
- removed the Ref** at (94.2, 104.9)
- removed the Ref** at (90.5, 93.2)
- removed the Ref** at (93.8, 93.7)
- removed the Ref** at (101.4, 104.9)
- removed the Ref** at (91.6, 93.4)
- removed the Ref** at (114.7, 96.8)
- removed the Ref** at (112.5, 96.5)
- removed the Ref** at (90.5, 107.0)
- removed the Ref** at (112.5, 107.0)
- removed the Ref** at (113.6, 107.0)
- removed the Ref** at (113.6, 96.7)
- removed the Ref** at (96.0, 98.9)
- removed the Ref** at (93.8, 107.0)
- removed the Ref** at (115.8, 97.0)
- removed the Ref** at (103.2, 98.9)
- removed the Ref** at (105.0, 98.9)
- removed the Ref** at (105.0, 104.9)
- removed the Ref** at (99.6, 104.9)
- removed the Ref** at (101.4, 98.9)
- removed the Ref** at (110.4, 104.9)
- removed the Ref** at (110.4, 98.9)
- removed the Ref** at (65.1, 90.2)
- removed the Ref** at (97.8, 98.9)
- removed the Ref** at (67.3, 90.5)
- removed the Ref** at (66.2, 90.3)
- removed the Ref** at (64.0, 90.0)
- removed the Ref** at (43.2, 86.9)
- removed the Ref** at (42.1, 86.7)
- removed the Ref** at (45.3, 87.2)
- removed the Ref** at (44.2, 87.1)
- removed the Ref** at (45.7, 84.9)
- removed the Ref** at (45.7, 78.9)
- removed the Ref** at (63.7, 84.9)
- removed the Ref** at (97.8, 104.9)
- removed the Ref** at (63.7, 78.9)
- removed the Ref** at (65.1, 76.7)
- removed the Ref** at (64.0, 76.7)
- removed the Ref** at (67.3, 76.7)
- removed the Ref** at (66.2, 76.7)
- removed the Ref** at (43.1, 76.8)
- removed the Ref** at (42.1, 76.7)
- removed the Ref** at (45.3, 76.8)
- removed the Ref** at (44.2, 76.8)
- removed the Ref** at (61.9, 78.9)
- removed the Ref** at (94.2, 98.9)
- removed the Ref** at (61.9, 84.9)
- removed the Ref** at (60.1, 84.9)
- removed the Ref** at (60.1, 78.9)
- removed the Ref** at (52.9, 78.9)
- removed the Ref** at (52.9, 84.9)
- removed the Ref** at (58.3, 84.9)
- removed the Ref** at (58.3, 78.9)
- removed the Ref** at (56.5, 84.9)
- removed the Ref** at (56.5, 78.9)
- removed the Ref** at (54.7, 78.9)
- removed the Ref** at (112.2, 104.9)
- removed the Ref** at (54.7, 84.9)
- removed the Ref** at (49.3, 78.9)
- removed the Ref** at (49.3, 84.9)
- removed the Ref** at (51.1, 78.9)
- removed the Ref** at (51.1, 84.9)
- removed the Ref** at (47.5, 78.9)
- removed the Ref** at (47.5, 84.9)
- removed the Ref** at (112.2, 98.9)
- removed the Ref** at (106.8, 98.9)
- added Ref**: Val**, kbd:IM_HOLE, F.Cu at (92.0, 93.3)
- added Ref**: Val**, kbd:IM_HOLE, F.Cu at (91.5, 93.3)
- added Ref**: Val**, kbd:IM_HOLE, F.Cu at (114.4, 107.1)
- added Ref**: Val**, kbd:IM_HOLE, F.Cu at (115.7, 107.1)
- added Ref**: Val**, kbd:IM_HOLE, F.Cu at (115.3, 107.1)
- added Ref**: Val**, kbd:IM_HOLE, F.Cu at (93.3, 93.5)
- added Ref**: Val**, kbd:IM_HOLE, F.Cu at (93.8, 93.6)
- added Ref**: Val**, kbd:IM_HOLE, F.Cu at (90.6, 93.1)
- added Ref**: Val**, kbd:IM_HOLE, F.Cu at (92.9, 93.5)
- added Ref**: Val**, kbd:IM_HOLE, F.Cu at (92.4, 93.4)
- added Ref**: Val**, kbd:IM_HOLE, F.Cu at (91.1, 93.2)
- added Ref**: Val**, kbd:IM_HOLE, F.Cu at (91.5, 107.1)
- added Ref**: Val**, kbd:IM_HOLE, F.Cu at (112.6, 107.1)
- added Ref**: Val**, kbd:IM_HOLE, F.Cu at (113.0, 107.1)
- added Ref**: Val**, kbd:IM_HOLE, F.Cu at (113.9, 107.1)
- added Ref**: Val**, kbd:IM_HOLE, F.Cu at (115.3, 96.8)
- added Ref**: Val**, kbd:IM_HOLE, F.Cu at (115.7, 96.9)
- added Ref**: Val**, kbd:IM_HOLE, F.Cu at (112.6, 96.4)
- added Ref**: Val**, kbd:IM_HOLE, F.Cu at (114.8, 107.1)
- added Ref**: Val**, kbd:IM_HOLE, F.Cu at (113.5, 107.1)
- added Ref**: Val**, kbd:IM_HOLE, F.Cu at (114.8, 96.7)
- added Ref**: Val**, kbd:IM_HOLE, F.Cu at (114.4, 96.7)
- added Ref**: Val**, kbd:IM_HOLE, F.Cu at (92.4, 107.1)
- added Ref**: Val**, kbd:IM_HOLE, F.Cu at (113.9, 96.6)
- added Ref**: Val**, kbd:IM_HOLE, F.Cu at (113.5, 96.5)
- added Ref**: Val**, kbd:IM_HOLE, F.Cu at (113.0, 96.5)
- added Ref**: Val**, kbd:IM_HOLE, F.Cu at (64.5, 90.2)
- added Ref**: Val**, kbd:IM_HOLE, F.Cu at (64.0, 90.2)
- added Ref**: Val**, kbd:IM_HOLE, F.Cu at (67.2, 90.6)
- added Ref**: Val**, kbd:IM_HOLE, F.Cu at (64.9, 90.3)
- added Ref**: Val**, kbd:IM_HOLE, F.Cu at (65.4, 90.3)
- added Ref**: Val**, kbd:IM_HOLE, F.Cu at (65.8, 90.4)
- added Ref**: Val**, kbd:IM_HOLE, F.Cu at (66.3, 90.5)
- added Ref**: Val**, kbd:IM_HOLE, F.Cu at (93.8, 107.1)
- added Ref**: Val**, kbd:IM_HOLE, F.Cu at (66.7, 90.6)
- added Ref**: Val**, kbd:IM_HOLE, F.Cu at (65.4, 76.6)
- added Ref**: Val**, kbd:IM_HOLE, F.Cu at (64.0, 76.6)
- added Ref**: Val**, kbd:IM_HOLE, F.Cu at (64.5, 76.6)
- added Ref**: Val**, kbd:IM_HOLE, F.Cu at (67.2, 76.6)
- added Ref**: Val**, kbd:IM_HOLE, F.Cu at (66.8, 76.6)
- added Ref**: Val**, kbd:IM_HOLE, F.Cu at (65.8, 76.6)
- added Ref**: Val**, kbd:IM_HOLE, F.Cu at (65.0, 76.6)
- added Ref**: Val**, kbd:IM_HOLE, F.Cu at (66.3, 76.6)
- added Ref**: Val**, kbd:IM_HOLE, F.Cu at (44.8, 87.3)
- added Ref**: Val**, kbd:IM_HOLE, F.Cu at (93.3, 107.1)
- added Ref**: Val**, kbd:IM_HOLE, F.Cu at (44.4, 87.2)
- added Ref**: Val**, kbd:IM_HOLE, F.Cu at (43.9, 87.2)
- added Ref**: Val**, kbd:IM_HOLE, F.Cu at (43.5, 87.1)
- added Ref**: Val**, kbd:IM_HOLE, F.Cu at (43.0, 87.0)
- added Ref**: Val**, kbd:IM_HOLE, F.Cu at (42.6, 87.0)
- added Ref**: Val**, kbd:IM_HOLE, F.Cu at (45.3, 87.4)
- added Ref**: Val**, kbd:IM_HOLE, F.Cu at (42.1, 86.9)
- added Ref**: Val**, kbd:IM_HOLE, F.Cu at (43.9, 76.6)
- added Ref**: Val**, kbd:IM_HOLE, F.Cu at (44.8, 76.6)
- added Ref**: Val**, kbd:IM_HOLE, F.Cu at (45.3, 76.6)
- added Ref**: Val**, kbd:IM_HOLE, F.Cu at (90.6, 107.1)
- added Ref**: Val**, kbd:IM_HOLE, F.Cu at (44.4, 76.6)
- added Ref**: Val**, kbd:IM_HOLE, F.Cu at (43.0, 76.6)
- added Ref**: Val**, kbd:IM_HOLE, F.Cu at (43.5, 76.6)
- added Ref**: Val**, kbd:IM_HOLE, F.Cu at (42.6, 76.6)
- added Ref**: Val**, kbd:IM_HOLE, F.Cu at (42.1, 76.6)
- added Ref**: Val**, kbd:IM_HOLE, F.Cu at (91.1, 107.1)
- added Ref**: Val**, kbd:IM_HOLE, F.Cu at (92.0, 107.1)
- added Ref**: Val**, kbd:IM_HOLE, F.Cu at (92.9, 107.1)
Connections:
- J2 pad 1: GND -> SDA
- J2 pad 2: VCC -> SCL
- J2 pad 3: SCL -> VCC
- J2 pad 4: SDA -> GND
- J7 pad 1: SDA_r -> GND
- J7 pad 2: SCL_r -> VCC
- J7 pad 3: VCC -> SCL_r
- J7 pad 4: GND -> SDA_r
Routing:
- net SDA_r: track 27.2 -> 35.9 mm, vias 0 -> 1
- net LED_r: track 53.6 -> 47.0 mm
- net SCL_r: track 23.9 -> 28.5 mm, vias 0 -> 1
- net SDA: track 24.9 -> 29.0 mm
- net VCC: track 377.1 -> 379.4 mm, vias 1 -> 3
- net Net-(D40-Pad2): track 13.5 -> 12.4 mm
- net Net-(D37-Pad2): track 12.1 -> 10.9 mm
- net Net-(D36-Pad2): track 12.1 -> 10.9 mm
- net Net-(D35-Pad2): track 12.1 -> 10.9 mm
- net Net-(D38-Pad2): track 12.1 -> 10.9 mm
- net Net-(D31-Pad2): track 12.1 -> 10.9 mm
- net Net-(D30-Pad2): track 12.1 -> 10.9 mm
- net Net-(D25-Pad2): track 12.1 -> 10.9 mm
- net Net-(D24-Pad2): track 12.1 -> 10.9 mm
- net Net-(D23-Pad2): track 12.1 -> 10.9 mm
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
Commit message: Update light
Parts:
- removed J10, J3, J5, J8: LED, kbd:StripLED_1side
- removed J4, J9: Conn_01x01, kbd:StripLED_OUT_1side
- D22, D23, D24, D25, D26, D27, D28, D29, D30, D31, D32, D33, D34, D35, D36, D37, D38, D39, D40, D41, D42: moved to B.Cu
Connections:
- J6 pad C: GND -> GNDA
- J6 pad D: VCC -> VDD
- J7 pad 1: GND -> GNDA
- J7 pad 2: VCC -> VDD
- RSW2 pad 2: GND -> GNDA
- U2 pad 21: VCC -> VDD
- U2 pad 23: GND -> GNDA
- U2 pad 3: GND -> GNDA
- U2 pad 4: GND -> GNDA
Routing:
- net VCC: track 379.4 -> 57.1 mm, vias 3 -> 0
- net LED: track 61.4 -> 0.00 mm
- net Net-(J4-Pad1): track 48.1 -> 0.00 mm
- net Net-(J10-Pad2): track 47.2 -> 0.00 mm, vias 2 -> 0
- net LED_r: track 47.0 -> 0.00 mm, vias 1 -> 0
- net VDD: track 0.00 -> 44.1 mm
- net col5_r: track 141.1 -> 139.1 mm
- added copper zone on B.Cu, net GNDA
- added copper zone on F.Cu, net GNDA

Commit message: corne-light-rev1.1.0
Parts:
- removed ? (x14): , kbd:LEGO_HOLE
- removed the G*** at (22.9, 143.2)
- removed the G*** at (134.7, 40.8)
- removed the Ref** at (92.0, 93.3)
- removed the Ref** at (91.5, 93.3)
- removed the Ref** at (114.4, 107.1)
- removed the Ref** at (115.7, 107.1)
- removed the Ref** at (115.3, 107.1)
- removed the Ref** at (93.3, 93.5)
- removed the Ref** at (93.8, 93.6)
- removed the Ref** at (90.6, 93.1)
- removed the Ref** at (92.9, 93.5)
- removed the Ref** at (92.4, 93.4)
- removed the Ref** at (91.1, 93.2)
- removed the Ref** at (91.5, 107.1)
- removed the Ref** at (112.6, 107.1)
- removed the Ref** at (113.0, 107.1)
- removed the Ref** at (113.9, 107.1)
- removed the Ref** at (115.3, 96.8)
- removed the Ref** at (115.7, 96.9)
- removed the Ref** at (112.6, 96.4)
- removed the Ref** at (114.8, 107.1)
- removed the Ref** at (113.5, 107.1)
- removed the Ref** at (114.8, 96.7)
- removed the Ref** at (114.4, 96.7)
- removed the Ref** at (92.4, 107.1)
- removed the Ref** at (113.9, 96.6)
- removed the Ref** at (113.5, 96.5)
- removed the Ref** at (113.0, 96.5)
- removed the Ref** at (64.5, 90.2)
- removed the Ref** at (64.0, 90.2)
- removed the Ref** at (67.2, 90.6)
- removed the Ref** at (64.9, 90.3)
- removed the Ref** at (65.4, 90.3)
- removed the Ref** at (65.8, 90.4)
- removed the Ref** at (66.3, 90.5)
- removed the Ref** at (93.8, 107.1)
- removed the Ref** at (66.7, 90.6)
- removed the Ref** at (65.4, 76.6)
- removed the Ref** at (64.0, 76.6)
- removed the Ref** at (64.5, 76.6)
- removed the Ref** at (67.2, 76.6)
- removed the Ref** at (66.8, 76.6)
- removed the Ref** at (65.8, 76.6)
- removed the Ref** at (65.0, 76.6)
- removed the Ref** at (66.3, 76.6)
- removed the Ref** at (44.8, 87.3)
- removed the Ref** at (93.3, 107.1)
- removed the Ref** at (44.4, 87.2)
- removed the Ref** at (43.9, 87.2)
- removed the Ref** at (43.5, 87.1)
- removed the Ref** at (43.0, 87.0)
- removed the Ref** at (42.6, 87.0)
- removed the Ref** at (45.3, 87.4)
- removed the Ref** at (42.1, 86.9)
- removed the Ref** at (43.9, 76.6)
- removed the Ref** at (44.8, 76.6)
- removed the Ref** at (45.3, 76.6)
- removed the Ref** at (90.6, 107.1)
- removed the Ref** at (44.4, 76.6)
- removed the Ref** at (43.0, 76.6)
- removed the Ref** at (43.5, 76.6)
- removed the Ref** at (42.6, 76.6)
- removed the Ref** at (42.1, 76.6)
- removed the Ref** at (91.1, 107.1)
- removed the Ref** at (92.0, 107.1)
- removed the Ref** at (92.9, 107.1)
- added G***: LOGO, kbd:corne-logo-silk, F.Cu at (279.3, 89.3)
- added G***: LOGO, kbd:corne-logo-silk, B.Cu at (279.3, 89.3)
- added G***: LOGO, kbd:corne-logo-silk, B.Cu at (18.0, 89.3)
- added G***: LOGO, kbd:corne-logo-silk, F.Cu at (18.0, 89.3)
- added J5: Breakaway_Tabs, locallib:breakaway-mousebites, F.Cu at (237.1, 93.1)
- added J5: Breakaway_Tabs, locallib:breakaway-mousebites, F.Cu at (275.2, 93.1)
- added J5: Breakaway_Tabs, locallib:breakaway-mousebites, F.Cu at (237.1, 32.2)
- added J5: Breakaway_Tabs, locallib:breakaway-mousebites, F.Cu at (199.1, 32.2)
- added J5: Breakaway_Tabs, locallib:breakaway-mousebites, F.Cu at (98.2, 32.2)
- added J5: Breakaway_Tabs, locallib:breakaway-mousebites, F.Cu at (60.2, 32.2)
- added J5: Breakaway_Tabs, locallib:breakaway-mousebites, F.Cu at (60.2, 93.0)
- added J5: Breakaway_Tabs, locallib:breakaway-mousebites, F.Cu at (22.2, 93.0)
- added Ref**: Val**, kbd:M2_Threads_v2, B.Cu at (144.4, 92.9)
- added Ref**: Val**, kbd:M2_HOLE_v2, F.Cu at (175.8, 99.3)
- added Ref**: Val**, kbd:M2_HOLE_v2, F.Cu at (222.4, 91.5)
- added Ref**: Val**, kbd:M2_HOLE_v2, F.Cu at (189.6, 51.8)
- added Ref**: Val**, kbd:M2_HOLE_v2, F.Cu at (265.5, 74.3)
- added Ref**: Val**, kbd:M2_HOLE_v2, F.Cu at (265.5, 55.3)
- added Ref**: Val**, kbd:M2_Threads_v2, B.Cu at (129.9, 84.4)
- added Ref**: Val**, kbd:M2_Threads_v2, F.Cu at (152.7, 92.9)
- added Ref**: Val**, kbd:M2_Threads_v2, F.Cu at (167.2, 84.4)
- added Ref**: Val**, kbd:M2_HOLE_v2, B.Cu at (121.4, 99.3)
- added Ref**: Val**, kbd:M2_HOLE_v2, B.Cu at (74.8, 91.7)
- added Ref**: Val**, kbd:M2_HOLE_v2, B.Cu at (31.7, 55.4)
- added Ref**: Val**, kbd:M2_HOLE_v2, B.Cu at (107.7, 51.9)
- added Ref**: Val**, kbd:M2_HOLE_v2, B.Cu at (31.7, 74.4)
- D22, D23, D24, D25, D26, D27, D28, D29, D30, D31, D32, D33, D34, D35, D36, D37, D38, D39, D40, D41, D42, J6, J7, RSW2: moved to F.Cu
- SW1, SW10, SW11, SW12, SW13, SW14, SW15, SW16, SW17, SW18, SW19, SW2, SW20, SW3, SW4, SW5, SW6, SW7, SW8, SW9: footprint kbd:CherryMX_Choc_1u -> kbd:CherryMX_1u
- SW21: footprint kbd:CherryMX_Choc_1.5u -> kbd:CherryMX_1u
- SW22, SW23, SW24, SW25, SW26, SW27, SW28, SW29, SW30, SW31, SW32, SW33, SW34, SW35, SW36, SW37, SW38, SW39, SW40, SW41: footprint kbd:CherryMX_Choc_1u -> kbd:CherryMX_1u; moved to F.Cu
- SW42: footprint kbd:CherryMX_Choc_1.5u -> kbd:CherryMX_1u; moved to F.Cu
- U1: footprint kbd:ProMicro_v2_1side -> kbd:ProMicro_v3
- U2: footprint kbd:ProMicro_v2_1side -> kbd:ProMicro_v3; moved to F.Cu
- moved D25 195.9 mm to (226.0, 40.8)
- moved D23 188.7 mm to (264.0, 45.8)
- moved SW25 185.0 mm to (218.0, 38.6), turned to 0 degrees
- moved D24 182.0 mm to (229.0, 40.8)
- moved D26 182.0 mm to (191.0, 40.8)
- moved D27 182.0 mm to (188.0, 40.8)
- moved SW24 181.9 mm to (237.0, 41.0), turned to 0 degrees
- moved SW26 181.9 mm to (199.0, 41.0), turned to 0 degrees
- moved SW27 178.8 mm to (180.0, 43.4), turned to 0 degrees
- moved SW22 175.8 mm to (275.0, 45.8), turned to 0 degrees
- moved SW23 175.8 mm to (256.0, 45.8), turned to 0 degrees
- moved D22 175.7 mm to (267.0, 45.8)
- moved D31 175.0 mm to (226.0, 59.8)
- moved D29 169.6 mm to (264.0, 64.8)
- moved U2 163.0 mm to (160.4, 56.5)
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Routing:
- net GNDA: track 0.09 -> 80.3 mm
- net reset_r: track 27.0 -> 89.3 mm
- net GND: track 12.6 -> 68.6 mm, vias 2 -> 0
- net col3_r: track 182.6 -> 135.6 mm, vias 0 -> 1
- net col1_r: track 196.9 -> 151.7 mm, vias 0 -> 1
- net col2_r: track 175.5 -> 130.3 mm, vias 0 -> 1
- net col4_r: track 161.7 -> 116.8 mm, vias 0 -> 1
- net col5_r: track 139.1 -> 95.1 mm, vias 0 -> 1
- net col0_r: track 221.0 -> 177.7 mm, vias 0 -> 1
- net row0_r: track 154.1 -> 113.6 mm
- net row0: track 165.8 -> 127.5 mm, vias 1 -> 0
- net data: track 43.3 -> 78.1 mm
- net col4: track 134.5 -> 105.1 mm, vias 0 -> 1
- net col3: track 151.0 -> 125.0 mm, vias 0 -> 1
- net row1_r: track 131.3 -> 112.6 mm
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- removed copper zone on B.Cu, net GND
- removed copper zone on F.Cu, net GND
- removed copper zone on B.Cu, net GNDA
- removed copper zone on F.Cu, net GNDA
Other:
- board size 133.8 x 157.4 mm -> 271.8 x 105.6 mm
- board text added: "Corne Light rev1.1.0 PCB Designed by foostan"
- board text removed: "Corne Light v2.1 PCB Designed by foostan"

Commit message: Update corne-right to rev1.1.1
Parts:
- added  : , locallib:breakaway-mousebites, F.Cu at (243.7, 117.4)
- added  : , locallib:breakaway-mousebites, F.Cu at (243.7, 105.4)
- added  : , locallib:breakaway-mousebites, F.Cu at (53.7, 117.5)
- added  : , locallib:breakaway-mousebites, F.Cu at (53.7, 105.5)
- added Ref**: Val**, kbd:M2_Threads_v2, F.Cu at (46.6, 108.5)
- added Ref**: Val**, kbd:M2_Threads_v2, F.Cu at (46.6, 114.5)
- added Ref**: Val**, kbd:M2_Threads_v2, F.Cu at (43.6, 120.5)
- added Ref**: Val**, kbd:M2_Threads_v2, F.Cu at (43.6, 114.5)
- added Ref**: Val**, kbd:M2_Threads_v2, F.Cu at (31.6, 120.5)
- added Ref**: Val**, kbd:M2_Threads_v2, F.Cu at (31.6, 114.5)
- added Ref**: Val**, kbd:M2_Threads_v2, F.Cu at (28.6, 120.5)
- added Ref**: Val**, kbd:M2_Threads_v2, F.Cu at (28.6, 114.5)
- added Ref**: Val**, kbd:M2_Threads_v2, F.Cu at (22.6, 120.5)
- added Ref**: Val**, kbd:M2_Threads_v2, F.Cu at (22.6, 108.5)
- added Ref**: Val**, kbd:M2_Threads_v2, F.Cu at (22.6, 102.5)
- added Ref**: Val**, kbd:M2_Threads_v2, F.Cu at (46.6, 102.5)
- added Ref**: Val**, kbd:M2_Threads_v2, F.Cu at (40.6, 114.5)
- added Ref**: Val**, kbd:M2_Threads_v2, F.Cu at (25.6, 120.5)
- added Ref**: Val**, kbd:M2_Threads_v2, F.Cu at (19.6, 120.5)
- added Ref**: Val**, kbd:M2_Threads_v2, F.Cu at (25.6, 114.5)
- added Ref**: Val**, kbd:M2_Threads_v2, F.Cu at (19.6, 114.5)
- added Ref**: Val**, kbd:M2_Threads_v2, F.Cu at (34.6, 120.5)
- added Ref**: Val**, kbd:M2_Threads_v2, F.Cu at (34.6, 114.5)
- added Ref**: Val**, kbd:M2_Threads_v2, F.Cu at (22.6, 114.5)
- added Ref**: Val**, kbd:M2_Threads_v2, F.Cu at (37.6, 120.5)
- added Ref**: Val**, kbd:M2_Threads_v2, F.Cu at (37.6, 114.5)
- added Ref**: Val**, kbd:M2_Threads_v2, F.Cu at (43.6, 108.5)
- added Ref**: Val**, kbd:M2_Threads_v2, F.Cu at (40.6, 120.5)
- added Ref**: Val**, kbd:M2_Threads_v2, F.Cu at (37.6, 108.5)
- added Ref**: Val**, kbd:M2_Threads_v2, F.Cu at (37.6, 102.5)
- added Ref**: Val**, kbd:M2_Threads_v2, F.Cu at (40.6, 108.5)
- added Ref**: Val**, kbd:M2_Threads_v2, F.Cu at (40.6, 102.5)
- added Ref**: Val**, kbd:M2_Threads_v2, F.Cu at (25.6, 108.5)
- added Ref**: Val**, kbd:M2_Threads_v2, F.Cu at (50.7, 117.4)
- added Ref**: Val**, kbd:M2_Threads_v2, F.Cu at (15.7, 105.5)
- added Ref**: Val**, kbd:M2_Threads_v2, F.Cu at (50.7, 105.4)
- added Ref**: Val**, kbd:M2_Threads_v2, F.Cu at (19.6, 108.5)
- added Ref**: Val**, kbd:M2_Threads_v2, F.Cu at (43.6, 102.5)
- added Ref**: Val**, kbd:M2_Threads_v2, F.Cu at (25.6, 102.5)
- added Ref**: Val**, kbd:M2_Threads_v2, F.Cu at (19.6, 102.5)
- added Ref**: Val**, kbd:M2_Threads_v2, F.Cu at (34.6, 108.5)
- added Ref**: Val**, kbd:M2_Threads_v2, F.Cu at (34.6, 102.5)
- added Ref**: Val**, kbd:M2_Threads_v2, F.Cu at (15.7, 117.5)
- added Ref**: Val**, kbd:M2_Threads_v2, F.Cu at (277.7, 120.5)
- added Ref**: Val**, kbd:M2_Threads_v2, F.Cu at (277.7, 114.5)
- added Ref**: Val**, kbd:M2_Threads_v2, F.Cu at (274.7, 120.5)
- added Ref**: Val**, kbd:M2_Threads_v2, F.Cu at (274.7, 114.5)
- added Ref**: Val**, kbd:M2_Threads_v2, F.Cu at (262.7, 120.5)
- added Ref**: Val**, kbd:M2_Threads_v2, F.Cu at (31.6, 108.5)
- added Ref**: Val**, kbd:M2_Threads_v2, F.Cu at (262.7, 114.5)
- added Ref**: Val**, kbd:M2_Threads_v2, F.Cu at (259.7, 120.5)
- added Ref**: Val**, kbd:M2_Threads_v2, F.Cu at (259.7, 114.5)
- added Ref**: Val**, kbd:M2_Threads_v2, F.Cu at (253.7, 120.5)
- added Ref**: Val**, kbd:M2_Threads_v2, F.Cu at (253.7, 114.5)
- added Ref**: Val**, kbd:M2_Threads_v2, F.Cu at (268.7, 120.5)
- added Ref**: Val**, kbd:M2_Threads_v2, F.Cu at (268.7, 114.5)
- added Ref**: Val**, kbd:M2_Threads_v2, F.Cu at (271.7, 120.5)
- added Ref**: Val**, kbd:M2_Threads_v2, F.Cu at (271.7, 114.5)
- added Ref**: Val**, kbd:M2_Threads_v2, F.Cu at (256.7, 120.5)
- added Ref**: Val**, kbd:M2_Threads_v2, F.Cu at (31.6, 102.5)
- added Ref**: Val**, kbd:M2_Threads_v2, F.Cu at (250.7, 120.5)
- added Ref**: Val**, kbd:M2_Threads_v2, F.Cu at (256.7, 114.5)
- added Ref**: Val**, kbd:M2_Threads_v2, F.Cu at (250.7, 114.5)
- added Ref**: Val**, kbd:M2_Threads_v2, F.Cu at (265.7, 120.5)
- added Ref**: Val**, kbd:M2_Threads_v2, F.Cu at (265.7, 114.5)
- added Ref**: Val**, kbd:M2_Threads_v2, F.Cu at (274.7, 108.5)
- added Ref**: Val**, kbd:M2_Threads_v2, F.Cu at (274.7, 102.5)
- added Ref**: Val**, kbd:M2_Threads_v2, F.Cu at (277.7, 108.5)
- added Ref**: Val**, kbd:M2_Threads_v2, F.Cu at (277.7, 102.5)
- added Ref**: Val**, kbd:M2_Threads_v2, F.Cu at (268.7, 108.5)
- added Ref**: Val**, kbd:M2_Threads_v2, F.Cu at (28.6, 108.5)
- added Ref**: Val**, kbd:M2_Threads_v2, F.Cu at (268.7, 102.5)
- added Ref**: Val**, kbd:M2_Threads_v2, F.Cu at (271.7, 108.5)
- added Ref**: Val**, kbd:M2_Threads_v2, F.Cu at (271.7, 102.5)
- added Ref**: Val**, kbd:M2_Threads_v2, F.Cu at (265.7, 108.5)
- added Ref**: Val**, kbd:M2_Threads_v2, F.Cu at (265.7, 102.5)
- added Ref**: Val**, kbd:M2_Threads_v2, F.Cu at (262.7, 108.5)
- added Ref**: Val**, kbd:M2_Threads_v2, F.Cu at (262.7, 102.5)
- added Ref**: Val**, kbd:M2_Threads_v2, F.Cu at (259.7, 108.5)
- added Ref**: Val**, kbd:M2_Threads_v2, F.Cu at (259.7, 102.5)
- added Ref**: Val**, kbd:M2_Threads_v2, F.Cu at (256.7, 108.5)
- added Ref**: Val**, kbd:M2_Threads_v2, F.Cu at (28.6, 102.5)
- added Ref**: Val**, kbd:M2_Threads_v2, F.Cu at (256.7, 102.5)
- added Ref**: Val**, kbd:M2_Threads_v2, F.Cu at (253.7, 108.5)
- added Ref**: Val**, kbd:M2_Threads_v2, F.Cu at (253.7, 102.5)
- added Ref**: Val**, kbd:M2_Threads_v2, F.Cu at (246.8, 117.5)
- added Ref**: Val**, kbd:M2_Threads_v2, F.Cu at (281.8, 117.4)
- added Ref**: Val**, kbd:M2_Threads_v2, F.Cu at (246.8, 105.5)
- added Ref**: Val**, kbd:M2_Threads_v2, F.Cu at (281.8, 105.4)
- added Ref**: Val**, kbd:M2_Threads_v2, F.Cu at (250.7, 108.5)
- added Ref**: Val**, kbd:M2_Threads_v2, F.Cu at (250.7, 102.5)
- added Ref**: Val**, kbd:M2_Threads_v2, F.Cu at (46.6, 120.5)
Routing:
- net SDA_r: track 29.7 -> 32.7 mm
- net SDA: track 29.7 -> 32.4 mm
- net row1: track 142.6 -> 145.0 mm
- net row0: track 127.5 -> 129.2 mm
- net SCL: track 28.2 -> 27.7 mm
Other:
- board size 271.8 x 105.6 mm -> 271.9 x 105.6 mm
- board text added: "Corne Light rev1.1.1 PCB Designed by foostan"
- board text removed: "Corne Light rev1.1.0 PCB Designed by foostan"
