File: corne-light/pcb/corne-light.kicad_pcb (KiCad board)
At the start: 2 copper layers, 271.9 x 105.6 mm, 210 parts, among them J1 MJ-4PP-9, J2 OLED, J5 Breakaway_Tabs, J6 MJ-4PP-9, J7 OLED, SW1 SW_PUSH, SW10 SW_PUSH, SW11 SW_PUSH, SW12 SW_PUSH, SW13 SW_PUSH, SW14 SW_PUSH, SW15 SW_PUSH, SW16 SW_PUSH, SW17 SW_PUSH, SW18 SW_PUSH, SW19 SW_PUSH, SW2 SW_PUSH, SW20 SW_PUSH, SW21 SW_PUSH, SW22 SW_PUSH, SW23 SW_PUSH, SW24 SW_PUSH, SW25 SW_PUSH, SW26 SW_PUSH, SW27 SW_PUSH, SW28 SW_PUSH, SW29 SW_PUSH, SW3 SW_PUSH, SW30 SW_PUSH, SW31 SW_PUSH, SW32 SW_PUSH, SW33 SW_PUSH, SW34 SW_PUSH, SW35 SW_PUSH, SW36 SW_PUSH, SW37 SW_PUSH, SW38 SW_PUSH, SW39 SW_PUSH, SW4 SW_PUSH, SW40 SW_PUSH, SW41 SW_PUSH, SW42 SW_PUSH, SW5 SW_PUSH, SW6 SW_PUSH, SW7 SW_PUSH, SW8 SW_PUSH, SW9 SW_PUSH, U1 ProMicro, U2 ProMicro

Commit message: Update light
Parts:
- removed  : , locallib:breakaway-mousebites (x4)
- removed the Ref** at (46.6, 108.5)
- removed the Ref** at (46.6, 114.5)
- removed the Ref** at (43.6, 120.5)
- removed the Ref** at (43.6, 114.5)
- removed the Ref** at (31.6, 120.5)
- removed the Ref** at (31.6, 114.5)
- removed the Ref** at (28.6, 120.5)
- removed the Ref** at (28.6, 114.5)
- removed the Ref** at (22.6, 120.5)
- removed the Ref** at (22.6, 108.5)
- removed the Ref** at (22.6, 102.5)
- removed the Ref** at (46.6, 102.5)
- removed the Ref** at (40.6, 114.5)
- removed the Ref** at (25.6, 120.5)
- removed the Ref** at (19.6, 120.5)
- removed the Ref** at (25.6, 114.5)
- removed the Ref** at (19.6, 114.5)
- removed the Ref** at (34.6, 120.5)
- removed the Ref** at (34.6, 114.5)
- removed the Ref** at (22.6, 114.5)
- removed the Ref** at (37.6, 120.5)
- removed the Ref** at (37.6, 114.5)
- removed the Ref** at (43.6, 108.5)
- removed the Ref** at (40.6, 120.5)
- removed the Ref** at (37.6, 108.5)
- removed the Ref** at (37.6, 102.5)
- removed the Ref** at (40.6, 108.5)
- removed the Ref** at (40.6, 102.5)
- removed the Ref** at (25.6, 108.5)
- removed the Ref** at (50.7, 117.4)
- removed the Ref** at (15.7, 105.5)
- removed the Ref** at (50.7, 105.4)
- removed the Ref** at (19.6, 108.5)
- removed the Ref** at (43.6, 102.5)
- removed the Ref** at (25.6, 102.5)
- removed the Ref** at (19.6, 102.5)
- removed the Ref** at (34.6, 108.5)
- removed the Ref** at (34.6, 102.5)
- removed the Ref** at (15.7, 117.5)
- removed the Ref** at (277.7, 120.5)
- removed the Ref** at (277.7, 114.5)
- removed the Ref** at (274.7, 120.5)
- removed the Ref** at (274.7, 114.5)
- removed the Ref** at (262.7, 120.5)
- removed the Ref** at (31.6, 108.5)
- removed the Ref** at (262.7, 114.5)
- removed the Ref** at (259.7, 120.5)
- removed the Ref** at (259.7, 114.5)
- removed the Ref** at (253.7, 120.5)
- removed the Ref** at (253.7, 114.5)
- removed the Ref** at (268.7, 120.5)
- removed the Ref** at (268.7, 114.5)
- removed the Ref** at (271.7, 120.5)
- removed the Ref** at (271.7, 114.5)
- removed the Ref** at (256.7, 120.5)
- removed the Ref** at (31.6, 102.5)
- removed the Ref** at (250.7, 120.5)
- removed the Ref** at (256.7, 114.5)
- removed the Ref** at (250.7, 114.5)
- removed the Ref** at (265.7, 120.5)
- removed the Ref** at (265.7, 114.5)
- removed the Ref** at (274.7, 108.5)
- removed the Ref** at (274.7, 102.5)
- removed the Ref** at (277.7, 108.5)
- removed the Ref** at (277.7, 102.5)
- removed the Ref** at (268.7, 108.5)
- removed the Ref** at (28.6, 108.5)
- removed the Ref** at (268.7, 102.5)
- removed the Ref** at (271.7, 108.5)
- removed the Ref** at (271.7, 102.5)
- removed the Ref** at (265.7, 108.5)
- removed the Ref** at (265.7, 102.5)
- removed the Ref** at (262.7, 108.5)
- removed the Ref** at (262.7, 102.5)
- removed the Ref** at (259.7, 108.5)
- removed the Ref** at (259.7, 102.5)
- removed the Ref** at (256.7, 108.5)
- removed the Ref** at (28.6, 102.5)
- removed the Ref** at (256.7, 102.5)
- removed the Ref** at (253.7, 108.5)
- removed the Ref** at (253.7, 102.5)
- removed the Ref** at (246.8, 117.5)
- removed the Ref** at (281.8, 117.4)
- removed the Ref** at (246.8, 105.5)
- removed the Ref** at (281.8, 105.4)
- removed the Ref** at (250.7, 108.5)
- removed the Ref** at (250.7, 102.5)
- removed the Ref** at (46.6, 120.5)
Other:
- board size 271.9 x 105.6 mm -> 271.8 x 105.6 mm

Commit message: fixed typo
Other:
- board text added: "Corne Light rev1.1.1 PCB designed by foostan"
- board text removed: "Corne Light rev1.1.1 PCB Designed by foostan"
Changed lines of the file:
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@@
   (gr_line (start 284.2745 127.439) (end 284.4145 127.267) (layer Edge.Cuts) (width 0.2))
   (gr_line (start 278.7125 94.625) (end 278.4815 94.602) (layer Edge.Cuts) (width 0.2))
-  (gr_text "Corne Light rev1.1.1\nPCB Designed by foostan" (at 246.014 90.594) (layer B.SilkS)
+  (gr_text "Corne Light rev1.1.1\nPCB designed by foostan" (at 246.014 90.594) (layer B.SilkS)
     (effects (font (size 1 1) (thickness 0.125)) (justify left mirror))
   )
-  (gr_text "Corne Light rev1.1.1\nPCB Designed by foostan" (at 226.654 90.564) (layer F.SilkS)
+  (gr_text "Corne Light rev1.1.1\nPCB designed by foostan" (at 226.654 90.564) (layer F.SilkS)
     (effects (font (size 1 1) (thickness 0.125)) (justify left))
   )
@@
   (gr_line (start 51.1968 36.6951) (end 51.1967 36.6952) (layer Edge.Cuts) (width 0.2))
   (gr_line (start 51.1969 36.6951) (end 51.1968 36.6951) (layer Edge.Cuts) (width 0.2))
-  (gr_text "Corne Light rev1.1.1\nPCB Designed by foostan" (at 70.44525 90.494) (layer B.SilkS)
+  (gr_text "Corne Light rev1.1.1\nPCB designed by foostan" (at 70.44525 90.494) (layer B.SilkS)
     (effects (font (size 1 1) (thickness 0.125)) (justify left mirror))
   )
-  (gr_text "Corne Light rev1.1.1\nPCB Designed by foostan" (at 51.08525 90.464) (layer F.SilkS)
+  (gr_text "Corne Light rev1.1.1\nPCB designed by foostan" (at 51.08525 90.464) (layer F.SilkS)
     (effects (font (size 1 1) (thickness 0.125)) (justify left))
   )

Commit message: Add kailh low profiile
Parts:
- SW1, SW10, SW11, SW12, SW13, SW14, SW15, SW16, SW17, SW18, SW19, SW2, SW20, SW22, SW23, SW24, SW25, SW26, SW27, SW28, SW29, SW3, SW30, SW31, SW32, SW33, SW34, SW35, SW36, SW37, SW38, SW39, SW4, SW40, SW41, SW5, SW6, SW7, SW8, SW9: footprint kbd:CherryMX_1u -> kbd:CherryMX_Choc_1u
- SW21, SW42: footprint kbd:CherryMX_1u -> kbd:CherryMX_Choc_1.5u
Routing:
- net col3: track 125.0 -> 140.9 mm
- net col2: track 120.1 -> 135.1 mm
- net col4_r: track 116.9 -> 131.4 mm
- net col3_r: track 135.8 -> 150.3 mm
- net col4: track 105.3 -> 118.6 mm
- net col5: track 92.3 -> 105.1 mm
- net Net-(D21-Pad2): track 33.6 -> 46.2 mm
- net col2_r: track 130.3 -> 142.9 mm
- net Net-(D41-Pad2): track 13.0 -> 25.5 mm
- net col5_r: track 95.3 -> 107.8 mm
- net Net-(D42-Pad2): track 31.8 -> 44.2 mm
- net col1: track 144.0 -> 156.4 mm
- net Net-(D16-Pad2): track 12.7 -> 25.0 mm
- net Net-(D37-Pad2): track 7.82 -> 20.1 mm
- net Net-(D8-Pad2): track 11.9 -> 24.1 mm
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Other:
- board text added: "Corne Light rev1.2 PCB Designed by foostan"
- board text removed: "Corne Light rev1.1.1 PCB designed by foostan"

Commit message: Update cuts and footprints
Parts:
- removed G*** (x4): LOGO, kbd:corne-logo-silk
- removed the Ref** at (175.8, 99.3)
- removed the Ref** at (222.4, 91.5)
- removed the Ref** at (189.6, 51.8)
- removed the Ref** at (265.5, 74.3)
- removed the Ref** at (265.5, 55.3)
- added Ref**: Val**, kbd:M2_Threads_v2, B.Cu at (269.2, 74.4)
- added Ref**: Val**, kbd:M2_Threads_v2, B.Cu at (269.2, 55.4)
- added Ref**: Val**, kbd:M2_Threads_v2, B.Cu at (226.1, 91.7)
- added Ref**: Val**, kbd:M2_Threads_v2, B.Cu at (179.5, 99.4)
- added Ref**: Val**, kbd:M2_Threads_v2, B.Cu at (193.2, 51.9)
- D1, D10, D11, D12, D13, D14, D15, D16, D17, D18, D19, D2, D20, D21, D22, D23, D24, D25, D26, D27, D28, D29, D3, D30, D31, D32, D33, D34, D35, D36, D37, D38, D39, D4, D40, D41, D42, D5, D6, D7, D8, D9: moved to B.Cu
- J5 (x8): footprint locallib:breakaway-mousebites -> kbd:Breakaway_Tabs
- Ref** (x5): footprint kbd:M2_HOLE_v2 -> kbd:M2_Threads_v2
- SW1, SW10, SW11, SW12, SW13, SW14, SW15, SW16, SW17, SW18, SW19, SW2, SW20, SW22, SW23, SW24, SW25, SW26, SW27, SW28, SW29, SW3, SW30, SW31, SW32, SW33, SW34, SW35, SW36, SW37, SW38, SW39, SW4, SW40, SW41, SW5, SW6, SW7, SW8, SW9: footprint kbd:CherryMX_Choc_1u -> kbd:CherryMX_ChocV2_1u
- SW21, SW42: footprint kbd:CherryMX_Choc_1.5u -> kbd:CherryMX_ChocV2_1.5u
- moved RSW2 3.76 mm to (156.4, 76.8)
- moved J6 3.76 mm to (154.6, 84.6)
- moved J5 3.69 mm to (240.8, 93.4)
- moved J5 3.68 mm to (278.8, 93.4)
- moved J5 3.67 mm to (240.8, 32.0)
- moved D22 3.66 mm to (270.7, 45.9)
- moved D23 3.66 mm to (267.7, 45.9)
- moved D24 3.66 mm to (232.7, 40.9)
- moved D25 3.66 mm to (229.7, 40.9)
- moved D26 3.66 mm to (194.7, 40.9)
- moved D27 3.66 mm to (191.7, 40.9)
- moved D28 3.66 mm to (270.7, 64.9)
- moved D29 3.66 mm to (267.7, 64.9)
- moved D30 3.66 mm to (232.7, 59.9)
- moved D31 3.66 mm to (229.7, 59.9)
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Routing:
- net row2_r: track 118.7 -> 131.5 mm
- net row3_r: track 78.4 -> 86.2 mm
- net row1_r: track 121.3 -> 129.1 mm
- net row0_r: track 116.8 -> 124.4 mm
- net row1: track 151.9 -> 155.9 mm
- net row3: track 93.2 -> 96.9 mm
- net row2: track 137.9 -> 141.0 mm
- net row0: track 131.5 -> 134.2 mm
- net GNDA: track 80.3 -> 78.1 mm
- net col5_r: track 107.8 -> 105.6 mm
- net GND: track 68.6 -> 66.6 mm
- net Net-(D27-Pad2): track 18.5 -> 20.5 mm
- net data_r: track 62.4 -> 64.4 mm
- net Net-(D21-Pad2): track 46.2 -> 48.2 mm
- net col0: track 182.2 -> 180.2 mm, vias 3 -> 1
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Other:
- board size 271.8 x 105.6 mm -> 275.5 x 105.6 mm

Commit message: Update libs of corne-light
Parts:
- moved J7 7.60 mm to (160.3, 77.3), turned to 0 degrees
Connections:
- net LED renamed Net-(U1-Pad1)
- net LED_r renamed Net-(U2-Pad1)
- J7 pad 1: GNDA -> SDA_r
- J7 pad 2: VDD -> SCL_r
- J7 pad 3: SCL_r -> VDD
- J7 pad 4: SDA_r -> GNDA
Other:
- board text added: "Corne Light v2.0 PCB Designed by foostan"
- board text removed: "Corne Light rev1.2 PCB Designed by foostan"
