File: corne-light/pcb/corne-light.sch (KiCad schematic (older format))
At the start: 98 parts, among them J1 MJ-4PP-9, J10 LED, J2 OLED, J3 LED, J4 Conn_01x01, J5 LED, J6 MJ-4PP-9, J7 OLED, J8 LED, J9 Conn_01x01, SW1 SW_PUSH, SW10 SW_PUSH, SW11 SW_PUSH, SW12 SW_PUSH, SW13 SW_PUSH, SW14 SW_PUSH, SW15 SW_PUSH, SW16 SW_PUSH, SW17 SW_PUSH, SW18 SW_PUSH, SW19 SW_PUSH, SW2 SW_PUSH, SW20 SW_PUSH, SW21 SW_PUSH, SW22 SW_PUSH, SW23 SW_PUSH, SW24 SW_PUSH, SW25 SW_PUSH, SW26 SW_PUSH, SW27 SW_PUSH, SW28 SW_PUSH, SW29 SW_PUSH, SW3 SW_PUSH, SW30 SW_PUSH, SW31 SW_PUSH, SW32 SW_PUSH, SW33 SW_PUSH, SW34 SW_PUSH, SW35 SW_PUSH, SW36 SW_PUSH, SW37 SW_PUSH, SW38 SW_PUSH, SW39 SW_PUSH, SW4 SW_PUSH, SW40 SW_PUSH, SW41 SW_PUSH, SW42 SW_PUSH, SW5 SW_PUSH, SW6 SW_PUSH, SW7 SW_PUSH, SW8 SW_PUSH, SW9 SW_PUSH, U1 ProMicro, U2 ProMicro

Commit message: Brashup righ hand
Connections:
- wire segments 122 -> 124
Changed lines of the file:
@@
 EESchema Schematic File Version 4
+LIBS:corne-light-cache
 EELAYER 26 0
 EELAYER END
@@
 $EndComp
 $Comp
-L power:GND #PWR019
-U 1 1 5A92390A
-P 5650 2800
-F 0 "#PWR019" H 5650 2550 50  0001 C CNN
-F 1 "GND" H 5650 2650 50  0000 C CNN
-F 2 "" H 5650 2800 50  0001 C CNN
-F 3 "" H 5650 2800 50  0001 C CNN
-	1    5650 2800
-	1    0    0    -1
-$EndComp
-$Comp
 L power:VCC #PWR018
 U 1 1 5A923DD7
-P 5775 2700
-F 0 "#PWR018" H 5775 2550 50  0001 C CNN
-F 1 "VCC" H 5775 2850 50  0000 C CNN
-F 2 "" H 5775 2700 50  0001 C CNN
-F 3 "" H 5775 2700 50  0001 C CNN
-	1    5775 2700
+P 6000 2600
+F 0 "#PWR018" H 6000 2450 50  0001 C CNN
+F 1 "VCC" H 6000 2750 50  0000 C CNN
+F 2 "" H 6000 2600 50  0001 C CNN
+F 3 "" H 6000 2600 50  0001 C CNN
+	1    6000 2600
 	0    1    1    0
 $EndComp
-Text GLabel 5650 2600 2    47   Input ~ 0
+Text GLabel 5650 2700 2    47   Input ~ 0
 SCL
-Text GLabel 5650 2500 2    47   Input ~ 0
+Text GLabel 5650 2800 2    47   Input ~ 0
 SDA
 $Comp
@@
 L power:GND #PWR0106
 U 1 1 5C25F9D8
-P 5950 5550
-F 0 "#PWR0106" H 5950 5300 50  0001 C CNN
-F 1 "GND" H 5950 5400 50  0000 C CNN
-F 2 "" H 5950 5550 50  0001 C CNN
-F 3 "" H 5950 5550 50  0001 C CNN
-	1    5950 5550
+P 5675 5725
+F 0 "#PWR0106" H 5675 5475 50  0001 C CNN
+F 1 "GND" H 5675 5575 50  0000 C CNN
+F 2 "" H 5675 5725 50  0001 C CNN
+F 3 "" H 5675 5725 50  0001 C CNN
+	1    5675 5725
 	1    0    0    -1
 $EndComp
@@
 L power:VCC #PWR0107
 U 1 1 5C25F9E4
-P 6025 5475
-F 0 "#PWR0107" H 6025 5325 50  0001 C CNN
-F 1 "VCC" H 6025 5625 50  0000 C CNN
-F 2 "" H 6025 5475 50  0001 C CNN
-F 3 "" H 6025 5475 50  0001 C CNN
-	1    6025 5475
+P 5750 5575
+F 0 "#PWR0107" H 5750 5425 50  0001 C CNN
+F 1 "VCC" H 5750 5725 50  0000 C CNN
+F 2 "" H 5750 5575 50  0001 C CNN
+F 3 "" H 5750 5575 50  0001 C CNN
+	1    5750 5575
 	0    1    1    0
 $EndComp
-Text GLabel 5600 5575 2    47   Input ~ 0
+Text GLabel 5600 5475 2    47   Input ~ 0
 SCL_r
-Text GLabel 5600 5675 2    47   Input ~ 0
+Text GLabel 5600 5375 2    47   Input ~ 0
 SDA_r
 $Comp
@@
 NoConn ~ 8325 1625
 NoConn ~ 8350 4875
-Wire Wire Line
-	5600 5375 5950 5375
-Wire Wire Line
-	5950 5375 5950 5550
-Wire Wire Line
-	5600 5475 6025 5475
-Wire Wire Line
-	5650 2700 5775 2700
 $Comp
 L Connector_Generic:Conn_01x03 J5
@@
 	-1   0    0    1
 $EndComp
+Wire Wire Line
+	5650 2600 6000 2600
+$Comp
+L power:GND #PWR019
+U 1 1 5A92390A
+P 5950 2675
+F 0 "#PWR019" H 5950 2425 50  0001 C CNN
+F 1 "GND" H 5950 2525 50  0000 C CNN
+F 2 "" H 5950 2675 50  0001 C CNN
+F 3 "" H 5950 2675 50  0001 C CNN
+	1    5950 2675
+	1    0    0    -1
+$EndComp
+Wire Wire Line
+	5950 2675 5950 2500
+Wire Wire Line
+	5950 2500 5650 2500
+Wire Wire Line
+	5600 5575 5750 5575
+Wire Wire Line
+	5600 5675 5675 5675
+Wire Wire Line
+	5675 5675 5675 5725
 $EndSCHEMATC

Commit message: Update light
Parts:
- removed J10, J3, J5, J8: LED, kbd:StripLED_1side, symbol Connector_Generic:Conn_01x03
- removed J4, J9: Conn_01x01, kbd:StripLED_OUT_1side, symbol Connector_Generic:Conn_01x01
Connections:
- net labels added: GNDA, VDD
- wire segments 124 -> 112

Commit message: Update cuts and footprints
Parts:
- U1, U2: symbol kbd:ProMicro -> corne-light-rescue:ProMicro-kbd
Connections:
- net GND: now also U1.23 (GND), U1.3 (GND), U1.4 (GND); no longer U1.1 (TX0/D3), U1.2 (RX1/D2)
- net GNDA: now also U2.23 (GND), U2.3 (GND), U2.4 (GND); no longer U2.1 (TX0/D3), U2.2 (RX1/D2)
- net LED: now also U1.1 (TX)
- net LED_r: now also U2.1 (TX)
- net SCL: now also U1.6 (SCL); no longer U1.4 (GND)
- net SCL_r: now also U2.6 (SCL); no longer U2.4 (GND)
- net SDA: now also U1.5 (SDA); no longer U1.3 (GND)
- net SDA_r: now also U2.5 (SDA); no longer U2.3 (GND)
- net VCC: now also U1.21 (VCC); no longer U1.23 (GND)
- net VDD: now also U2.21 (VCC); no longer U2.23 (GND)
- net col0: now also U1.20 (F4); no longer U1.22 (RST)
- net col0_r: now also U2.20 (F4); no longer U2.22 (RST)
- net col1: now also U1.19 (F5); no longer U1.21 (VCC)
- net col1_r: now also U2.19 (F5); no longer U2.21 (VCC)
- net col2: now also U1.18 (F6); no longer U1.20 (F4/A3)
- net col2_r: now also U2.18 (F6); no longer U2.20 (F4/A3)
- net col3: now also U1.17 (F7); no longer U1.19 (F5/A2)
- net col3_r: now also U2.17 (F7); no longer U2.19 (F5/A2)
- net col4: now also U1.16 (B1); no longer U1.18 (F6/A1)
- net col4_r: now also U2.16 (B1); no longer U2.18 (F6/A1)
- net col5: now also U1.15 (B3); no longer U1.17 (F7/A0)
- net col5_r: now also U2.15 (B3); no longer U2.17 (F7/A0)
- net data: now also U1.2 (RX)
- net data_r: now also U2.2 (RX)
- net reset: now also U1.22 (RST); no longer U1.24 (RAW)
- net reset_r: now also U2.22 (RST); no longer U2.24 (RAW)
- net row0: now also U1.7 (D4); no longer U1.5 (2/D1/SDA)
- net row0_r: now also U2.7 (D4); no longer U2.5 (2/D1/SDA)
- net row1: now also U1.8 (C6); no longer U1.6 (3/D0/SCL)
- net row1_r: now also U2.8 (C6); no longer U2.6 (3/D0/SCL)
- net row2: now also U1.9 (D7); no longer U1.7 (4/D4)
- net row2_r: now also U2.9 (D7); no longer U2.7 (4/D4)
- net row3: now also U1.10 (E6); no longer U1.8 (5/C6)
- net row3_r: now also U2.10 (E6); no longer U2.8 (5/C6)
Other:
- moved on the sheet: U1, U2
Changed lines of the file:
@@
 EESchema Schematic File Version 4
-LIBS:corne-light-cache
-EELAYER 26 0
+EELAYER 30 0
 EELAYER END
 $Descr A4 11693 8268
@@
 $EndDescr
 $Comp
-L kbd:ProMicro U1
+L corne-light-rescue:ProMicro-kbd U1
 U 1 1 5A5E14C2
 P 6225 1625
@@
 	4125 2150 4125 2750
 $Comp
-L kbd:ProMicro U2
+L corne-light-rescue:ProMicro-kbd U2
 U 1 1 5C25F857
 P 6225 4500

Commit message: Update libs of corne-light
Parts:
- SW1, SW10, SW11, SW12, SW13, SW14, SW15, SW16, SW17, SW18, SW19, SW2, SW20, SW22, SW23, SW24, SW25, SW26, SW27, SW28, SW29, SW3, SW30, SW31, SW32, SW33, SW34, SW35, SW36, SW37, SW38, SW39, SW4, SW40, SW41, SW5, SW6, SW7, SW8, SW9: footprint kbd:CherryMX_Choc_1u -> kbd:CherryMX_ChocV2_1u
- SW21, SW42: footprint kbd:CherryMX_Choc_1.5u -> kbd:CherryMX_ChocV2_1.5u
- U1, U2: footprint kbd:ProMicro_v2_1side -> kbd:ProMicro_v3; symbol corne-light-rescue:ProMicro-kbd -> kbd:ProMicro
Connections:
- net GNDA: now also J7.4 (Pin_4); no longer J7.1 (Pin_1)
- net SCL_r: now also J7.2 (Pin_2); no longer J7.3 (Pin_3)
- net SDA_r: now also J7.1 (Pin_1); no longer J7.4 (Pin_4)
- net VDD: now also J7.3 (Pin_3); no longer J7.2 (Pin_2)
- net LED: no longer names the net of U1.1 (TX0/D3)
- net LED_r: no longer names the net of U2.1 (TX0/D3)
- no-connect marks 12 -> 15
