File: corne-light/pcb_top/corne-top-plate.kicad_pcb (KiCad board)
At the start: 2 copper layers, 132.9 x 91.4 mm, 26 parts, among them SW2 KEY_SWITCH

Commit message: fixed typo
Other:
- board text added: "Corne Keyboard PCB designed by foostan"
- board text removed: "Corne Keyboard PCB Designed by foostan"
Changed lines of the file:
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@@
   (gr_line (start 155.51 83) (end 155.5 83) (angle 90) (layer Eco2.User) (width 2.5))
   (gr_line (start 79.5 105.5) (end 79.51 105.5) (angle 90) (layer Eco2.User) (width 2.5))
-  (gr_text "Corne Keyboard\nPCB Designed by foostan" (at 118.406 121.741) (layer B.SilkS)
+  (gr_text "Corne Keyboard\nPCB designed by foostan" (at 118.406 121.741) (layer B.SilkS)
     (effects (font (size 1 1) (thickness 0.125)) (justify left mirror))
   )
-  (gr_text "Corne Keyboard\nPCB Designed by foostan" (at 99.036 121.741) (layer F.SilkS)
+  (gr_text "Corne Keyboard\nPCB designed by foostan" (at 99.036 121.741) (layer F.SilkS)
     (effects (font (size 1 1) (thickness 0.125)) (justify left))
   )
