File: corne-cherry/pcb/corne-cherry.sch (KiCad schematic (older format))
At the start: 87 parts, among them J1 MJ-4PP-9, J2 OLED, J3 LED, P1 i2c-pin, P2 i2c-pin, SW1 SW_PUSH, SW10 SW_PUSH, SW11 SW_PUSH, SW12 SW_PUSH, SW13 SW_PUSH, SW14 SW_PUSH, SW15 SW_PUSH, SW16 SW_PUSH, SW17 SW_PUSH, SW18 SW_PUSH, SW19 SW_PUSH, SW2 SW_PUSH, SW20 SW_PUSH, SW21 SW_PUSH, SW3 SW_PUSH, SW4 SW_PUSH, SW5 SW_PUSH, SW6 SW_PUSH, SW7 SW_PUSH, SW8 SW_PUSH, SW9 SW_PUSH, U1 ProMicro

Commit message: Update corne-cherry
Parts:
- D1, D10, D11, D12, D13, D14, D15, D16, D17, D18, D19, D2, D20, D21, D3, D4, D5, D6, D7, D8, D9: symbol D -> Device:D
- J1: symbol MJ-4PP-9 -> kbd:MJ-4PP-9
- J2: symbol Conn_01x04 -> Connector_Generic:Conn_01x04
- J3: symbol Conn_01x03 -> Connector_Generic:Conn_01x03
- JP1: symbol Jumper -> Device:Jumper
- JP2, JP3, JP4, JP5, JP6, JP7, JP8, JP9: symbol Jumper_NO_Small -> Device:Jumper_NO_Small
- L1, L10, L11, L12, L13, L14, L15, L16, L17, L18, L19, L2, L20, L21, L22, L23, L24, L25, L26, L27, L3, L4, L5, L6, L7, L8, L9: symbol SK6812MINI -> kbd:SK6812MINI
- P1, P2: symbol Conn_01x01 -> Connector_Generic:Conn_01x01
- R1, R2: symbol R -> Device:R
- RSW1, SW1, SW10, SW11, SW12, SW13, SW14, SW15, SW16, SW17, SW18, SW19, SW2, SW20, SW21, SW3, SW4, SW5, SW6, SW7, SW8, SW9: symbol SW_PUSH -> kbd:SW_PUSH
- U1: symbol ProMicro -> kbd:ProMicro

Commit message: Update footprints
Parts:
- U1: symbol kbd:ProMicro -> corne-cherry-rescue:ProMicro-kbd
Changed lines of the file:
@@
 EESchema Schematic File Version 4
-LIBS:corne-cherry-cache
-EELAYER 26 0
+EELAYER 30 0
 EELAYER END
 $Descr A4 11693 8268
@@
 $EndDescr
 $Comp
-L kbd:ProMicro U1
+L corne-cherry-rescue:ProMicro-kbd U1
 U 1 1 5A5E14C2
 P 1800 1950

Commit message: Update corne cherry to v3.0
Parts:
- removed J3: LED, kbd:StripLED_rev, symbol Connector_Generic:Conn_01x03
- removed JP1: (no value), kbd:JPC2, symbol Device:Jumper
- removed JP2, JP3, JP4, JP5, JP6, JP7, JP8, JP9: (no value), kbd:Jumper, symbol Device:Jumper_NO_Small
- removed L1, L10, L11, L12, L13, L14, L15, L16, L17, L18, L19, L2, L20, L21, L3, L4, L5, L6, L7, L8, L9: SK6812MINI, kbd:SK6812MINI_rev, symbol kbd:SK6812MINI
- removed L22, L23, L24, L25, L26, L27: SK6812MINI, kbd:SK6812MINI_underglow, symbol kbd:SK6812MINI
- removed P1, P2: i2c-pin, kbd:1pin_conn, symbol Connector_Generic:Conn_01x01
- removed R1, R2: R, kbd:R, symbol Device:R
- added D22, D23, D24, D25, D26, D27, D28, D29, D30, D31, D32, D33, D34, D35, D36, D37, D38, D39, D40, D41, D42: D, kbd:D3_SMD_v2, symbol Device:D
- added J3: MJ-4PP-9, kbd:MJ-4PP-9_1side, symbol kbd:MJ-4PP-9
- added J4: OLED, kbd:OLED_1side, symbol Connector_Generic:Conn_01x04
- added LED1, LED2, LED28, LED29, LED3, LED30, LED31, LED32, LED33, LED4, LED5, LED6: WS2812B, LED_SMD:LED_WS2812B_PLCC4_5.0x5.0mm_P3.2mm, symbol LED:WS2812B
- added LED10, LED11, LED12, LED13, LED14, LED15, LED16, LED17, LED18, LED19, LED20, LED21, LED22, LED23, LED24, LED25, LED26, LED27, LED34, LED35, LED36, LED37, LED38, LED39, LED40, LED41, LED42, LED43, LED44, LED45, LED46, LED47, LED48, LED49, LED50, LED51, LED52, LED53, LED54, LED7, LED8, LED9: YS-SK6812MINI-E, kbd:YS-SK6812MINI-E, symbol kbd:YS-SK6812MINI-E
- added RSW2: SW_PUSH, kbd:ResetSW_1side, symbol kbd:SW_PUSH
- added SW22, SW23, SW24, SW25, SW26, SW27, SW28, SW29, SW30, SW31, SW32, SW33, SW34, SW35, SW36, SW37, SW38, SW39, SW40, SW41: SW_PUSH, kbd:CherryMX_Hotswap, symbol kbd:SW_PUSH
- added SW42: SW_PUSH, kbd:CherryMX_Hotswap_1.5u, symbol kbd:SW_PUSH
- added U2: ProMicro, kbd:ProMicro_v2_1side, symbol kbd:ProMicro
- D1, D10, D11, D12, D13, D14, D15, D16, D17, D18, D19, D2, D20, D21, D3, D4, D5, D6, D7, D8, D9: footprint kbd:D3_TH_SMD -> kbd:D3_SMD_v2
- J1: footprint kbd:MJ-4PP-9 -> kbd:MJ-4PP-9_1side
- J2: footprint kbd:OLED -> kbd:OLED_1side
- RSW1: footprint kbd:ResetSW -> kbd:ResetSW_1side
- SW1, SW10, SW11, SW12, SW13, SW14, SW15, SW16, SW17, SW18, SW19, SW2, SW20, SW3, SW4, SW5, SW6, SW7, SW8, SW9: footprint kbd:MX_ALPS_PG1350_noLed -> kbd:CherryMX_Hotswap
- SW21: footprint kbd:MX_ALPS_PG1350_noLed_1.75u -> kbd:CherryMX_Hotswap_1.5u
- U1: footprint kbd:ProMicro_v2 -> kbd:ProMicro_v2_1side; symbol corne-cherry-rescue:ProMicro-kbd -> kbd:ProMicro
Connections:
- net labels added: GNDA, LED_r, SCL_r, SDA_r, VDD, col0_r, col1_r, col2_r, col3_r, col4_r, col5_r, data_r, reset_r, row0_r, row1_r, row2_r, row3_r
- wire segments 265 -> 338
- no-connect marks 6 -> 14
Other:
- moved on the sheet: D1, D10, D11, D12, D13, D14, D15, D16, D17, D18, D19, D2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
