File: corne-cherry/pcb/corne-cherry.sch (KiCad schematic (older format))
At the start: 146 parts, among them J1 MJ-4PP-9, J2 OLED, J3 MJ-4PP-9, J4 OLED, SW1 SW_PUSH, SW10 SW_PUSH, SW11 SW_PUSH, SW12 SW_PUSH, SW13 SW_PUSH, SW14 SW_PUSH, SW15 SW_PUSH, SW16 SW_PUSH, SW17 SW_PUSH, SW18 SW_PUSH, SW19 SW_PUSH, SW2 SW_PUSH, SW20 SW_PUSH, SW21 SW_PUSH, SW22 SW_PUSH, SW23 SW_PUSH, SW24 SW_PUSH, SW25 SW_PUSH, SW26 SW_PUSH, SW27 SW_PUSH, SW28 SW_PUSH, SW29 SW_PUSH, SW3 SW_PUSH, SW30 SW_PUSH, SW31 SW_PUSH, SW32 SW_PUSH, SW33 SW_PUSH, SW34 SW_PUSH, SW35 SW_PUSH, SW36 SW_PUSH, SW37 SW_PUSH, SW38 SW_PUSH, SW39 SW_PUSH, SW4 SW_PUSH, SW40 SW_PUSH, SW41 SW_PUSH, SW42 SW_PUSH, SW5 SW_PUSH, SW6 SW_PUSH, SW7 SW_PUSH, SW8 SW_PUSH, SW9 SW_PUSH, U1 ProMicro, U2 ProMicro

Commit message: Update sch
Parts:
- U1, U2: footprint kbd:ProMicro_v2_1side -> kbd:ProMicro_v3
Changed lines of the file:
@@
 Sheet 1 1
 Title "Corne Cherry"
-Date "2020-07-20"
-Rev "3.0"
+Date "2020-09-28"
+Rev "3.0.1"
 Comp "foostan"
 Comment1 ""
@@
 F 0 "U1" H 1775 2675 60  0000 C CNN
 F 1 "ProMicro" H 1775 1175 60  0000 C CNN
-F 2 "kbd:ProMicro_v2_1side" H 1875 675 60  0001 C CNN
+F 2 "kbd:ProMicro_v3" H 1875 675 60  0001 C CNN
 F 3 "" H 1875 675 60  0000 C CNN
 	1    1775 1725
@@
 F 0 "U2" H 10175 2625 60  0000 C CNN
 F 1 "ProMicro" H 10175 1125 60  0000 C CNN
-F 2 "kbd:ProMicro_v2_1side" H 10275 625 60  0001 C CNN
+F 2 "kbd:ProMicro_v3" H 10275 625 60  0001 C CNN
 F 3 "" H 10275 625 60  0000 C CNN
 	1    10175 1675
@@
 L power:GNDA #PWR024
 U 1 1 5C25F9D8
-P 9425 3225
-F 0 "#PWR024" H 9425 2975 50  0001 C CNN
-F 1 "GNDA" H 9425 3075 50  0000 C CNN
-F 2 "" H 9425 3225 50  0001 C CNN
-F 3 "" H 9425 3225 50  0001 C CNN
-	1    9425 3225
-	1    0    0    -1
-$EndComp
-Text GLabel 9350 2975 2    47   Input ~ 0
+P 9725 3050
+F 0 "#PWR024" H 9725 2800 50  0001 C CNN
+F 1 "GNDA" H 9725 2900 50  0000 C CNN
+F 2 "" H 9725 3050 50  0001 C CNN
+F 3 "" H 9725 3050 50  0001 C CNN
+	1    9725 3050
+	1    0    0    -1
+$EndComp
+Text GLabel 9350 3075 2    47   Input ~ 0
 SCL_r
-Text GLabel 9350 2875 2    47   Input ~ 0
+Text GLabel 9350 3175 2    47   Input ~ 0
 SDA_r
 NoConn ~ 10875 1125
@@
 Wire Wire Line
 	1325 2775 1025 2775
-Wire Wire Line
-	9350 3075 9500 3075
-Wire Wire Line
-	9350 3175 9425 3175
-Wire Wire Line
-	9425 3175 9425 3225
 $Comp
 L power:VDD #PWR019
@@
 L power:VDD #PWR023
 U 1 1 5C71DE62
-P 9500 3075
-F 0 "#PWR023" H 9500 2925 50  0001 C CNN
-F 1 "VDD" V 9517 3203 50  0000 L CNN
-F 2 "" H 9500 3075 50  0001 C CNN
-F 3 "" H 9500 3075 50  0001 C CNN
-	1    9500 3075
+P 9800 2975
+F 0 "#PWR023" H 9800 2825 50  0001 C CNN
+F 1 "VDD" V 9817 3103 50  0000 L CNN
+F 2 "" H 9800 2975 50  0001 C CNN
+F 3 "" H 9800 2975 50  0001 C CNN
+	1    9800 2975
 	0    1    1    0
 $EndComp
@@
 	1    0    0    -1
 $EndComp
+Wire Wire Line
+	9350 2975 9800 2975
+Wire Wire Line
+	9350 2875 9725 2875
+Wire Wire Line
+	9725 2875 9725 3050
 $EndSCHEMATC
