File: corne-classic/pcb/corne-classic.sch (KiCad schematic (older format))
At the start: 87 parts, among them J1 MJ-4PP-9, J2 OLED, J3 LED, P1 i2c-pin, P2 i2c-pin, SW1 SW_PUSH, SW10 SW_PUSH, SW11 SW_PUSH, SW12 SW_PUSH, SW13 SW_PUSH, SW14 SW_PUSH, SW15 SW_PUSH, SW16 SW_PUSH, SW17 SW_PUSH, SW18 SW_PUSH, SW19 SW_PUSH, SW2 SW_PUSH, SW20 SW_PUSH, SW21 SW_PUSH, SW3 SW_PUSH, SW4 SW_PUSH, SW5 SW_PUSH, SW6 SW_PUSH, SW7 SW_PUSH, SW8 SW_PUSH, SW9 SW_PUSH, U1 ProMicro

Commit message: Rename crkbd to corne classic and some fix
Parts:
- D1, D10, D11, D12, D13, D14, D15, D16, D17, D18, D19, D2, D20, D21, D3, D4, D5, D6, D7, D8, D9: symbol D -> Device:D
- J1: symbol MJ-4PP-9 -> kbd:MJ-4PP-9
- J2: symbol Conn_01x04 -> Connector_Generic:Conn_01x04
- J3: symbol Conn_01x03 -> Connector_Generic:Conn_01x03
- JP1: footprint kbd:JPC2 -> kbd:JP; symbol Jumper -> Device:Jumper
- JP2, JP3, JP4, JP5, JP6, JP7, JP8, JP9: symbol Jumper_NO_Small -> Device:Jumper_NO_Small
- L1: renamed from L22; symbol SK6812MINI -> kbd:SK6812MINI
- L10: renamed from L4; symbol SK6812MINI -> kbd:SK6812MINI
- L11: renamed from L5; symbol SK6812MINI -> kbd:SK6812MINI
- L12: renamed from L6; symbol SK6812MINI -> kbd:SK6812MINI
- L13: renamed from L7; symbol SK6812MINI -> kbd:SK6812MINI
- L14: renamed from L8; symbol SK6812MINI -> kbd:SK6812MINI
- L15: renamed from L9; symbol SK6812MINI -> kbd:SK6812MINI
- L16: renamed from L10; symbol SK6812MINI -> kbd:SK6812MINI
- L17: renamed from L11; symbol SK6812MINI -> kbd:SK6812MINI
- L18: renamed from L12; symbol SK6812MINI -> kbd:SK6812MINI
- L19: renamed from L13; symbol SK6812MINI -> kbd:SK6812MINI
- L2: renamed from L23; symbol SK6812MINI -> kbd:SK6812MINI
- L20: renamed from L14; symbol SK6812MINI -> kbd:SK6812MINI
- L21: renamed from L15; symbol SK6812MINI -> kbd:SK6812MINI
- L22: renamed from L16; symbol SK6812MINI -> kbd:SK6812MINI
- L23: renamed from L17; symbol SK6812MINI -> kbd:SK6812MINI
- L24: renamed from L18; symbol SK6812MINI -> kbd:SK6812MINI
- L25: renamed from L19; symbol SK6812MINI -> kbd:SK6812MINI
- L26: renamed from L20; symbol SK6812MINI -> kbd:SK6812MINI
- L27: renamed from L21; symbol SK6812MINI -> kbd:SK6812MINI
- L3: renamed from L24; symbol SK6812MINI -> kbd:SK6812MINI
- L4: renamed from L25; symbol SK6812MINI -> kbd:SK6812MINI
- L5: renamed from L26; symbol SK6812MINI -> kbd:SK6812MINI
- L6: renamed from L27; symbol SK6812MINI -> kbd:SK6812MINI
- L7: renamed from L1; symbol SK6812MINI -> kbd:SK6812MINI
- L8: renamed from L2; symbol SK6812MINI -> kbd:SK6812MINI
- L9: renamed from L3; symbol SK6812MINI -> kbd:SK6812MINI
- P1, P2: symbol Conn_01x01 -> Connector_Generic:Conn_01x01
- R1, R2: symbol R -> Device:R
- RSW1, SW1, SW10, SW11, SW12, SW13, SW14, SW15, SW16, SW17, SW18, SW19, SW2, SW20, SW21, SW3, SW4, SW5, SW6, SW7, SW8, SW9: symbol SW_PUSH -> kbd:SW_PUSH
- U1: symbol ProMicro -> kbd:ProMicro
Connections:
- wire segments 184 -> 265

Commit message: Update refs in pcbnew
Changed lines of the file:
@@
 EESchema Schematic File Version 4
+LIBS:corne-classic-cache
 EELAYER 26 0
 EELAYER END
@@
 Text GLabel 5850 2550 0    60   Input ~ 0
 row2
-Text GLabel 7950 3150 0    60   Input ~ 0
+Text GLabel 7925 3150 0    60   Input ~ 0
 row3
 $Comp
@@
 	1350 4600 1350 4750
 Wire Wire Line
-	7950 3150 8100 3150
-Wire Wire Line
 	5850 2550 6000 2550
 Wire Wire Line
@@
 	6425 6175 6425 6325
 Wire Wire Line
-	6425 6325 5825 6325
-Wire Wire Line
-	5825 6325 5825 6175
-Wire Wire Line
 	8325 6475 8225 6475
 Wire Wire Line
@@
 	6525 6675 6525 6825
 Wire Wire Line
-	6525 6175 6525 6675
-Wire Wire Line
 	6525 5975 6525 6175
 Wire Wire Line
@@
 Wire Wire Line
 	8900 2250 8900 2850
+Wire Wire Line
+	6425 6325 5825 6325
+Wire Wire Line
+	5825 6175 5825 6325
+Wire Wire Line
+	7925 3150 8100 3150
+Wire Wire Line
+	6525 6175 6525 6675
 $EndSCHEMATC

Commit message: added libraries to folder, changes footprint associations
Parts:
- added D22: D, kbd:D3_TH_SMD, symbol Device:D
- added RV11: JOYSTICK-PSP1000, HackPack_Footprints:JOYSTICK-PSP1000, symbol arina:JOYSTICK-PSP1000
- added SW19: SW_PUSH, kailh-pg1425-x-switch:MX-ALPS-Choc-X-straight-crane, symbol corne-classic-rescue:SW_PUSH-kbd
- J1: symbol kbd:MJ-4PP-9 -> corne-classic-rescue:MJ-4PP-9-kbd
- L1, L10, L11, L12, L13, L14, L15, L16, L17, L18, L19, L2, L20, L21, L22, L23, L24, L25, L26, L27, L3, L4, L5, L6, L7, L8, L9: symbol kbd:SK6812MINI -> corne-classic-rescue:SK6812MINI-kbd
- RSW1: symbol kbd:SW_PUSH -> corne-classic-rescue:SW_PUSH-kbd
- SW1, SW10, SW11, SW12, SW13, SW14, SW15, SW16, SW17, SW18, SW2, SW3, SW4, SW5, SW6, SW7, SW8, SW9: footprint kbd:MX_ALPS_PG1350_noLed -> kailh-pg1425-x-switch:MX-ALPS-Choc-X-straight-crane; symbol kbd:SW_PUSH -> corne-classic-rescue:SW_PUSH-kbd
- SW20: renamed from SW19; footprint kbd:MX_ALPS_PG1350_noLed -> kailh-pg1425-x-switch:MX-ALPS-Choc-X-straight-crane; symbol kbd:SW_PUSH -> corne-classic-rescue:SW_PUSH-kbd
- SW21: renamed from SW20; footprint kbd:MX_ALPS_PG1350_noLed -> kailh-pg1425-x-switch:MX-ALPS-Choc-X-straight-crane; symbol kbd:SW_PUSH -> corne-classic-rescue:SW_PUSH-kbd
- SW22: renamed from SW21; footprint kbd:MX_ALPS_PG1350_noLed_1.75u -> kailh-pg1425-x-switch:MX-ALPS-Choc-X-straight-crane; symbol kbd:SW_PUSH -> corne-classic-rescue:SW_PUSH-kbd
- U1: symbol kbd:ProMicro -> corne-classic-rescue:ProMicro-kbd
Connections:
- net labels added: analogX, analogY
- wire segments 265 -> 272
- no-connect marks 6 -> 4

Commit message: reverted corne classic to original, made new folder
Parts:
- removed D22: D, kbd:D3_TH_SMD, symbol Device:D
- removed RV11: JOYSTICK-PSP1000, HackPack_Footprints:JOYSTICK-PSP1000, symbol arina:JOYSTICK-PSP1000
- removed SW19: SW_PUSH, kailh-pg1425-x-switch:MX-ALPS-Choc-X-straight-crane, symbol corne-classic-rescue:SW_PUSH-kbd
- J1: symbol corne-classic-rescue:MJ-4PP-9-kbd -> kbd:MJ-4PP-9
- L1, L10, L11, L12, L13, L14, L15, L16, L17, L18, L19, L2, L20, L21, L22, L23, L24, L25, L26, L27, L3, L4, L5, L6, L7, L8, L9: symbol corne-classic-rescue:SK6812MINI-kbd -> kbd:SK6812MINI
- RSW1: symbol corne-classic-rescue:SW_PUSH-kbd -> kbd:SW_PUSH
- SW1, SW10, SW11, SW12, SW13, SW14, SW15, SW16, SW17, SW18, SW2, SW3, SW4, SW5, SW6, SW7, SW8, SW9: footprint kailh-pg1425-x-switch:MX-ALPS-Choc-X-straight-crane -> kbd:MX_ALPS_PG1350_noLed; symbol corne-classic-rescue:SW_PUSH-kbd -> kbd:SW_PUSH
- SW19: renamed from SW20; footprint kailh-pg1425-x-switch:MX-ALPS-Choc-X-straight-crane -> kbd:MX_ALPS_PG1350_noLed; symbol corne-classic-rescue:SW_PUSH-kbd -> kbd:SW_PUSH
- SW20: renamed from SW21; footprint kailh-pg1425-x-switch:MX-ALPS-Choc-X-straight-crane -> kbd:MX_ALPS_PG1350_noLed; symbol corne-classic-rescue:SW_PUSH-kbd -> kbd:SW_PUSH
- SW21: renamed from SW22; footprint kailh-pg1425-x-switch:MX-ALPS-Choc-X-straight-crane -> kbd:MX_ALPS_PG1350_noLed_1.75u; symbol corne-classic-rescue:SW_PUSH-kbd -> kbd:SW_PUSH
- U1: symbol corne-classic-rescue:ProMicro-kbd -> kbd:ProMicro
Connections:
- net labels removed: analogX, analogY
- wire segments 272 -> 265
- no-connect marks 4 -> 6
