File: pcb/corne.kicad_pcb (KiCad board)
At the start: 2 copper layers, 275.5 x 105.6 mm, 172 parts, among them J1 MJ-4PP-9, J2 OLED, J3 MJ-4PP-9, J4 OLED, SW1 SW_PUSH, SW10 SW_PUSH, SW11 SW_PUSH, SW12 SW_PUSH, SW13 SW_PUSH, SW14 SW_PUSH, SW15 SW_PUSH, SW16 SW_PUSH, SW17 SW_PUSH, SW18 SW_PUSH, SW19 SW_PUSH, SW2 SW_PUSH, SW20 SW_PUSH, SW21 SW_PUSH, SW22 SW_PUSH, SW23 SW_PUSH, SW24 SW_PUSH, SW25 SW_PUSH, SW26 SW_PUSH, SW27 SW_PUSH, SW28 SW_PUSH, SW29 SW_PUSH, SW3 SW_PUSH, SW30 SW_PUSH, SW31 SW_PUSH, SW32 SW_PUSH, SW33 SW_PUSH, SW34 SW_PUSH, SW35 SW_PUSH, SW36 SW_PUSH, SW37 SW_PUSH, SW38 SW_PUSH, SW39 SW_PUSH, SW4 SW_PUSH, SW40 SW_PUSH, SW41 SW_PUSH, SW42 SW_PUSH, SW5 SW_PUSH, SW6 SW_PUSH, SW7 SW_PUSH, SW8 SW_PUSH, SW9 SW_PUSH, U1 ProMicro, U2 ProMicro

Commit message: Update pcb
Parts:
- removed D22, D23, D24, D25, D26, D27, D28, D29, D30, D31, D32, D33, D34, D35, D36, D37, D38, D39, D40, D41, D42: D, kbd:D3_SMD_v2
- removed G*** (x4): LOGO, kbd:corne-logo-horizontal
- removed LED22, LED23, LED24, LED25, LED26, LED27, LED34, LED35, LED36, LED37, LED38, LED39, LED40, LED41, LED42, LED43, LED44, LED45, LED46, LED47, LED48, LED49, LED50, LED51, LED52, LED53, LED54: YS-SK6812MINI-E, kbd:YS-SK6812MINI-E
- removed LED28, LED29, LED30, LED31, LED32, LED33: WS2812B, LED_SMD:LED_WS2812B_PLCC4_5.0x5.0mm_P3.2mm
- removed REF** (x8): Breakaway_Tabs, kbd:Breakaway_Tabs
- removed RSW1, RSW2: SW_PUSH, kbd:ResetSW_1side
- removed Ref** (x14): Val**, kbd:M2_HOLE_v2
- removed SW22, SW23, SW24, SW25, SW26, SW27, SW28, SW29, SW30, SW31, SW32, SW33, SW34, SW35, SW36, SW37, SW38, SW39, SW40, SW41: SW_PUSH, kbd_local:keyswitch_cherrymx_hotswap_1u
- removed SW42: SW_PUSH, kbd_local:keyswitch_cherrymx_hotswap_1.5u
- added C1: 20p, Capacitor_SMD:C_0603_1608Metric, B.Cu at (99.2, 102.2)
- added C10: 100n, Capacitor_SMD:C_0603_1608Metric, B.Cu at (82.9, 95.6)
- added C11: 10u, Capacitor_SMD:C_0603_1608Metric, B.Cu at (134.0, 99.1)
- added C12: 100n, Capacitor_SMD:C_0603_1608Metric, B.Cu at (86.8, 96.3)
- added C13: 100n, Capacitor_SMD:C_0603_1608Metric, B.Cu at (89.1, 87.0)
- added C14: 100n, Capacitor_SMD:C_0603_1608Metric, B.Cu at (86.8, 90.3)
- added C15: 100n, Capacitor_SMD:C_0603_1608Metric, B.Cu at (89.8, 93.8)
- added C16: 1u, Capacitor_SMD:C_0603_1608Metric, B.Cu at (112.0, 90.1)
- added C2: 20p, Capacitor_SMD:C_0603_1608Metric, B.Cu at (98.3, 110.2)
- added C3: 100n, Capacitor_SMD:C_0603_1608Metric, B.Cu at (89.2, 97.8)
- added C4: 100n, Capacitor_SMD:C_0603_1608Metric, B.Cu at (92.1, 96.3)
- added C5: 1u, Capacitor_SMD:C_0603_1608Metric, B.Cu at (89.8, 100.4)
- added C6: 10u, Capacitor_SMD:C_0603_1608Metric, B.Cu at (148.9, 100.3)
- added C7: 100n, Capacitor_SMD:C_0603_1608Metric, B.Cu at (92.1, 88.8)
- added C8: 1u, Capacitor_SMD:C_0603_1608Metric, B.Cu at (90.3, 91.2)
- added C9: 100n, Capacitor_SMD:C_0603_1608Metric, B.Cu at (86.6, 93.2)
- added EXD1: D, Diode_SMD:D_0603_1608Metric, B.Cu at (162.2, 57.6)
- added EXD2: D, Diode_SMD:D_0603_1608Metric, B.Cu at (162.2, 76.6)
- added EXLED1: YS-SK6812MINI-E, kbd_local:YS-SK6812MINI-E, B.Cu at (156.4, 64.8)
- added EXLED2: YS-SK6812MINI-E, kbd_local:YS-SK6812MINI-E, B.Cu at (156.4, 83.9)
- added EXSW1: RotaryEncoder_Switch, kbd_local:keyswitch_cherrymx_hotswap_1u_rotary_encoder_ec12, F.Cu at (156.4, 60.1)
- added EXSW2: RotaryEncoder_Switch, kbd_local:keyswitch_cherrymx_hotswap_1u_rotary_encoder_ec12, F.Cu at (156.4, 79.1)
- added F1: BSMD0603-050-12V, Fuse:Fuse_0603_1608Metric, B.Cu at (160.4, 51.3)
- added J5: Conn_01x06, Connector_PinHeader_2.54mm:PinHeader_1x06_P2.54mm_Vertical, F.Cu at (146.5, 73.1)
- added J6: Conn_01x06, Connector_PinHeader_2.54mm:PinHeader_1x06_P2.54mm_Vertical, F.Cu at (146.4, 52.8)
- added R1: 5.1k, Resistor_SMD:R_0603_1608Metric, B.Cu at (153.2, 51.2)
- added R2: 5.1k, Resistor_SMD:R_0603_1608Metric, B.Cu at (163.9, 51.0)
- added R3: 1k, Resistor_SMD:R_0603_1608Metric, B.Cu at (93.6, 102.1)
- added R4: 27, Resistor_SMD:R_0603_1608Metric, B.Cu at (150.0, 49.6)
- added R5: 27, Resistor_SMD:R_0603_1608Metric, B.Cu at (146.6, 49.5)
- added R6: 1k, Resistor_SMD:R_0603_1608Metric, B.Cu at (108.3, 89.6)
- added R7: 10k, Resistor_SMD:R_0603_1608Metric, B.Cu at (107.2, 86.5)
- added SMDSW1: SKQGADE010, Button_Switch_SMD:SW_SPST_SKQG_WithStem, B.Cu at (89.8, 74.1)
- added SMDSW2: SKQGADE010, Button_Switch_SMD:SW_SPST_SKQG_WithStem, B.Cu at (115.6, 96.4)
- added U3: TPD4E05U06DQAR, Package_SON:USON-10_2.5x1.0mm_P0.5mm, B.Cu at (148.4, 46.5)
- added U4: W25Q128JVSIQ, Package_SON:WSON-8-1EP_6x5mm_P1.27mm_EP3.4x4.3mm, B.Cu at (107.3, 95.0)
- added Y1: 12MHz 10pF, Crystal:Crystal_SMD_2520-4Pin_2.5x2.0mm, B.Cu at (96.6, 106.1)
- added ZD1: ESD5Z5V0C, Diode_SMD:D_SOD-523, B.Cu at (149.4, 51.9)
- D1, D10, D11, D12, D13, D14, D15, D16, D17, D18, D19, D2, D20, D21, D3, D4, D5, D6, D7, D8, D9: footprint kbd:D3_SMD_v2 -> Diode_SMD:D_0603_1608Metric
- J1: value MJ-4PP-9 -> TYPE-C-31-M-13C; footprint kbd:MJ-4PP-9_1side -> kbd_local:TYPE-C-31-M-13C; moved to B.Cu
- J2: value OLED -> ST-0277D00-052-142; footprint kbd:OLED_1side -> kbd_local:ST-0277D00-052-142
- J3: value MJ-4PP-9 -> Conn_01x04; footprint kbd:MJ-4PP-9_1side -> kbd_local:OLED
- J4: value OLED -> Conn_01x03; footprint kbd:OLED_1side -> Connector_PinHeader_2.54mm:PinHeader_1x03_P2.54mm_Vertical
- LED1, LED2, LED3, LED4, LED5, LED6: value WS2812B -> YS-SK6812MINI-E; footprint LED_SMD:LED_WS2812B_PLCC4_5.0x5.0mm_P3.2mm -> kbd_local:YS-SK6812MINI-E
- LED10, LED11, LED12, LED13, LED14, LED15, LED16, LED17, LED18, LED19, LED20, LED21, LED7, LED8, LED9: footprint kbd:YS-SK6812MINI-E -> kbd_local:YS-SK6812MINI-E
- SW1: value SW_PUSH -> SW_Push; footprint kbd_local:keyswitch_cherrymx_hotswap_1u -> kbd:keyswitch_cherrymx_hotswap_1.5u
- SW10, SW11, SW12, SW13, SW14, SW15, SW16, SW17, SW18, SW19, SW2, SW20, SW3, SW4, SW5, SW6, SW7, SW8, SW9: value SW_PUSH -> SW_Push; footprint kbd_local:keyswitch_cherrymx_hotswap_1u -> kbd:keyswitch_cherrymx_hotswap_1u
- SW21: value SW_PUSH -> SW_Push; footprint kbd_local:keyswitch_cherrymx_hotswap_1.5u -> kbd:keyswitch_cherrymx_hotswap_1u
- U1: value ProMicro -> RP2040; footprint kbd:ProMicro_v3 -> Package_DFN_QFN:QFN-56-1EP_7x7mm_P0.4mm_EP3.2x3.2mm; moved to B.Cu
- U2: value ProMicro -> NCP1117LPST33T3G; footprint kbd:ProMicro_v3 -> Package_TO_SOT_SMD:SOT-223-3_TabPin2; moved to B.Cu
- moved SW1 151.8 mm to (151.4, 111.9), turned to 66.12 degrees
- moved D1 142.1 mm to (151.5, 105.6), turned to -113.88 degrees
- moved LED1 135.3 mm to (155.8, 113.9), turned to -113.88 degrees
- moved LED8 116.1 mm to (128.6, 114.5), turned to 168.06 degrees
- moved SW2 111.5 mm to (137.3, 88.6)
- moved LED7 110.4 mm to (118.3, 91.0), turned to 180 degrees
- moved D2 108.8 mm to (143.2, 86.2), turned to 180 degrees
- moved SW8 105.9 mm to (129.6, 109.9), turned to -11.94 degrees
- moved D8 104.1 mm to (135.8, 108.7), turned to 168.06 degrees
- moved SW7 103.1 mm to (118.3, 86.2)
- moved D7 100.6 mm to (124.1, 83.8), turned to 180 degrees
- moved LED4 98.6 mm to (137.3, 55.3)
- moved LED9 91.9 mm to (108.7, 112.4), turned to 180 degrees
- moved J4 90.9 mm to (72.5, 97.5), turned to 90 degrees
- moved SW3 88.1 mm to (137.3, 69.6)
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Connections:
- D1 pad 1: row0 -> /ROW3
- D10 pad 1: row1 -> /ROW2
- D11 pad 1: row1 -> /ROW1
- D12 pad 1: row1 -> /ROW0
- D13 pad 1: row2 -> /ROW0
- D14 pad 1: row2 -> /ROW1
- D15 pad 1: row2 -> /ROW2
- D16 pad 1: row2 -> /ROW2
- D17 pad 1: row2 -> /ROW1
- D18 pad 1: row2 -> /ROW0
- D19 pad 1: row3 -> unconnected-(D19-K-Pad1)
- D19 pad 2: Net-(D19-Pad2) -> unconnected-(D19-A-Pad2)
- D2 pad 1: row0 -> /ROW2
- D20 pad 1: row3 -> /ROW1
- D21 pad 1: row3 -> /ROW2
- D3 pad 1: row0 -> /ROW1
- D4 pad 1: row0 -> /ROW0
- D4 pad 2: Net-(D4-Pad2) -> unconnected-(D4-A-Pad2)
- D5 pad 1: row0 -> /ROW0
- D6 pad 1: row0 -> /ROW1
- D6 pad 2: Net-(D6-Pad2) -> unconnected-(D6-A-Pad2)
- D7 pad 1: row1 -> /ROW2
- D8 pad 1: row1 -> /ROW3
- D9 pad 1: row1 -> /ROW3
- J4 pad 1: SDA_r -> /SWCLK
- J4 pad 2: SCL_r -> GND
- J4 pad 3: VDD -> /SWD
- LED1 pad 1: VCC -> +5V
- LED1 pad 2: Net-(LED1-Pad2) -> Net-(LED1-DOUT)
- LED1 pad 4: Net-(LED1-Pad4) -> /LED
- LED10 pad 1: VCC -> +5V
- LED10 pad 2: Net-(LED10-Pad2) -> Net-(LED10-DOUT)
- LED10 pad 4: Net-(LED10-Pad4) -> Net-(LED10-DIN)
- LED11 pad 1: VCC -> +5V
- LED11 pad 2: Net-(LED11-Pad2) -> Net-(LED11-DOUT)
- LED11 pad 4: Net-(LED11-Pad4) -> Net-(LED10-DOUT)
- LED12 pad 1: VCC -> +5V
- LED12 pad 2: Net-(LED11-Pad4) -> Net-(LED12-DOUT)
- LED12 pad 4: Net-(LED12-Pad4) -> Net-(LED11-DOUT)
- LED13 pad 1: VCC -> +5V
- LED13 pad 2: Net-(LED13-Pad2) -> Net-(LED13-DOUT)
- LED13 pad 4: Net-(LED13-Pad4) -> Net-(LED12-DOUT)
- LED14 pad 1: VCC -> +5V
- LED14 pad 2: Net-(LED14-Pad2) -> Net-(LED14-DOUT)
- LED14 pad 4: Net-(LED14-Pad4) -> Net-(LED13-DOUT)
- LED15 pad 1: VCC -> +5V
- LED15 pad 2: Net-(LED15-Pad2) -> Net-(LED15-DOUT)
- LED15 pad 4: Net-(LED15-Pad4) -> Net-(LED14-DOUT)
- LED16 pad 1: VCC -> +5V
- LED16 pad 2: Net-(LED10-Pad4) -> Net-(LED16-DOUT)
- LED16 pad 4: Net-(LED16-Pad4) -> Net-(LED15-DOUT)
- LED17 pad 1: VCC -> +5V
- LED17 pad 2: Net-(LED17-Pad2) -> Net-(LED17-DOUT)
- LED17 pad 4: Net-(LED11-Pad2) -> Net-(LED16-DOUT)
- LED18 pad 1: VCC -> +5V
- LED18 pad 2: Net-(LED12-Pad4) -> Net-(LED18-DOUT)
- LED18 pad 4: Net-(LED18-Pad4) -> Net-(LED17-DOUT)
- LED19 pad 1: VCC -> +5V
- LED19 pad 2: Net-(LED19-Pad2) -> Net-(LED19-DOUT)
- LED19 pad 4: Net-(LED13-Pad2) -> Net-(LED18-DOUT)
- LED2 pad 1: VCC -> +5V
- LED2 pad 2: Net-(LED1-Pad4) -> Net-(LED2-DOUT)
- LED2 pad 4: Net-(LED2-Pad4) -> Net-(LED1-DOUT)
- LED20 pad 1: VCC -> +5V
- LED20 pad 2: Net-(LED14-Pad4) -> Net-(LED20-DOUT)
- LED20 pad 4: Net-(LED20-Pad4) -> Net-(LED19-DOUT)
- LED21 pad 1: VCC -> +5V
- LED21 pad 2: Net-(LED20-Pad4) -> Net-(EXLED1-DIN)
- LED21 pad 4: Net-(LED15-Pad2) -> Net-(LED20-DOUT)
- LED3 pad 1: VCC -> +5V
- LED3 pad 2: Net-(LED2-Pad4) -> Net-(LED3-DOUT)
- LED3 pad 4: LED -> Net-(LED2-DOUT)
- LED4 pad 1: VCC -> +5V
- LED4 pad 4: Net-(LED1-Pad2) -> Net-(LED3-DOUT)
- LED5 pad 1: VCC -> +5V
- LED6 pad 1: VCC -> +5V
- LED6 pad 2: Net-(LED27-Pad4) -> Net-(LED6-DOUT)
- LED7 pad 1: VCC -> +5V
- LED7 pad 2: Net-(LED13-Pad4) -> Net-(LED7-DOUT)
- LED7 pad 4: Net-(LED7-Pad4) -> Net-(LED6-DOUT)
- LED8 pad 1: VCC -> +5V
- LED8 pad 2: Net-(LED7-Pad4) -> Net-(LED8-DOUT)
- LED8 pad 4: Net-(LED14-Pad2) -> Net-(LED7-DOUT)
- LED9 pad 1: VCC -> +5V
- LED9 pad 2: Net-(LED15-Pad4) -> Net-(LED10-DIN)
- LED9 pad 4: Net-(LED10-Pad2) -> Net-(LED8-DOUT)
- SW1 pad 1: col0 -> /COL5
- SW10 pad 1: col3 -> /COL3
- SW11 pad 1: col4 -> /COL3
- SW12 pad 1: col5 -> /COL3
- SW13 pad 1: col0 -> /COL2
- SW14 pad 1: col1 -> /COL2
- SW15 pad 1: col2 -> /COL2
- SW16 pad 1: col3 -> /COL1
- SW17 pad 1: col4 -> /COL1
- SW18 pad 1: col5 -> /COL1
- SW19 pad 1: col3 -> /COL0
- SW19 pad 2: Net-(D19-Pad2) -> unconnected-(SW19-Pad2)
- SW2 pad 1: col1 -> /COL5
- SW20 pad 1: col4 -> /COL0
- SW21 pad 1: col5 -> /COL0
- SW3 pad 1: col2 -> /COL5
- SW4 pad 1: col3 -> unconnected-(SW4-Pad1)
- SW4 pad 2: Net-(D4-Pad2) -> unconnected-(SW4-Pad2)
- SW5 pad 1: col4 -> /COL4
- SW6 pad 1: col5 -> unconnected-(SW6-Pad1)
- SW6 pad 2: Net-(D6-Pad2) -> unconnected-(SW6-Pad2)
- SW7 pad 1: col0 -> /COL4
- SW8 pad 1: col1 -> /COL4
- SW9 pad 1: col2 -> /COL3
- U1 pad 1: LED -> +3V3
- U1 pad 10: row3 -> +3V3
- U1 pad 11: Net-(U1-Pad11) -> /COL4
- U1 pad 12: Net-(U1-Pad12) -> /COL5
- U1 pad 13: Net-(U1-Pad13) -> /COL6
- U1 pad 14: Net-(U1-Pad14) -> /ROW0
- U1 pad 15: col5 -> /ROW1
- U1 pad 16: col4 -> /ROW2
- U1 pad 17: col3 -> /ROW3
- U1 pad 18: col2 -> unconnected-(U1-GPIO15-Pad18)
- U1 pad 19: col1 -> GND
- U1 pad 2: data -> /TX
- U1 pad 20: col0 -> Net-(U1-XIN)
- U1 pad 21: VCC -> Net-(U1-XOUT)
- U1 pad 22: reset -> +3V3
- U1 pad 23: GND -> +1V1
- U1 pad 24: Net-(U1-Pad24) -> /SWCLK
- U1 pad 3: GND -> /RX
- U1 pad 4: GND -> /SDA
- U1 pad 5: SDA -> /SCL
- U1 pad 6: SCL -> /COL0
- U1 pad 7: row0 -> /COL1
- U1 pad 8: row1 -> /COL2
- U1 pad 9: row2 -> /COL3
- U2 pad 1: LED_r -> GND
- U2 pad 2: data_r -> +3V3
- U2 pad 3: GNDA -> +5V
Routing:
- net GND: track 637.2 -> 0.00 mm, vias 16 -> 0
- net GNDA: track 617.9 -> 0.00 mm, vias 15 -> 0
- net VDD: track 573.1 -> 0.00 mm, vias 2 -> 0
- net VCC: track 544.3 -> 0.00 mm, vias 2 -> 0
- net row1: track 193.3 -> 0.00 mm, vias 2 -> 0
- net row0_r: track 184.4 -> 0.00 mm, vias 2 -> 0
- net row0: track 183.2 -> 0.00 mm, vias 2 -> 0
- net row2: track 180.7 -> 0.00 mm, vias 2 -> 0
- net col0_r: track 175.8 -> 0.00 mm, vias 5 -> 0
- net row2_r: track 172.6 -> 0.00 mm, vias 2 -> 0
- net col0: track 170.3 -> 0.00 mm, vias 5 -> 0
- net row1_r: track 166.9 -> 0.00 mm
- net col1_r: track 150.7 -> 0.00 mm, vias 5 -> 0
- net col1: track 149.4 -> 0.00 mm, vias 5 -> 0
- net col3_r: track 133.0 -> 0.00 mm, vias 7 -> 0
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Other:
- board size 275.5 x 105.6 mm -> 134.3 x 93.5 mm
- board text removed: "Corne Cherry v3.0.1 PCB Designed by foostan"

Commit message: Update pcb
Parts:
- J2: moved to B.Cu
- moved J5 76.9 mm to (70.3, 63.3)
- moved J6 57.9 mm to (89.3, 62.0)
- moved SMDSW1 18.5 mm to (108.3, 74.5)
- turned J2 to 90 degrees
Other:
- board text added: "Next: Change reset sqitch"
Changed lines of the file:
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@@
   )
   (footprint "Connector_PinHeader_2.54mm:PinHeader_1x06_P2.54mm_Vertical" (layer "F.Cu")
-    (at 146.52 73.0925)
+    (at 70.26 63.3425)
     (descr "Through hole straight pin header, 1x06, 2.54mm pitch, single row")
     (tags "Through hole pin header THT 1x06 2.54mm single row")
@@
   )
   (footprint "Connector_PinHeader_2.54mm:PinHeader_1x06_P2.54mm_Vertical" (layer "F.Cu")
-    (at 146.39 52.8225)
+    (at 89.26 62.0225)
     (descr "Through hole straight pin header, 1x06, 2.54mm pitch, single row")
     (tags "Through hole pin header THT 1x06 2.54mm single row")
@@
     )
   )
-  (footprint "kbd_local:ST-0277D00-052-142" (layer "F.Cu")
-    (at 166.68 94.2125 -90)
-    (descr "USB Type-C receptacle for USB 2.0 and PD, http://www.krhro.com/uploads/soft/180320/1-1P320120243.pdf")
-    (tags "usb usb-c 2.0 pd")
-    (property "JLCPCB Part #" "C2837093")
-    (property "Sheetfile" "corne.kicad_sch")
-    (property "Sheetname" "")
-    (property "ki_description" "Audio Jack, 4 Poles (TRRS)")
-    (property "ki_keywords" "audio jack receptacle stereo headphones TRRS connector")
-    (attr smd)
-    (fp_text reference "J2" (at 0 14.65 90) (layer "F.SilkS")
-        (effects (font (size 1 1) (thickness 0.15)))
-    )
-    (fp_text value "ST-0277D00-052-142" (at 0 16.2 90) (layer "F.Fab")
-        (effects (font (size 1 1) (thickness 0.15)))
-    )
-    (fp_line (start -3.35 0) (end -6 0)
-      (stroke (width 0.1) (type solid)) (layer "Edge.Cuts"))
-    (fp_line (start -3.35 0) (end -3.35 13.5)
-      (stroke (width 0.1) (type solid)) (layer "Edge.Cuts"))
-    (fp_line (start -3.35 13.5) (end 3.35 13.5)
-      (stroke (width 0.1) (type solid)) (layer "Edge.Cuts"))
-    (fp_line (start 3.35 0) (end 3.35 13.5)
-      (stroke (width 0.1) (type solid)) (layer "Edge.Cuts"))
-    (fp_line (start 6 0) (end 3.35 0)
-      (stroke (width 0.1) (type solid)) (layer "Edge.Cuts"))
-    (pad "R1" thru_hole oval (at 4.05 6 270) (size 0.75 1.8) (drill oval 0.45 1.5) (layers "*.Cu" "*.Mask")
-      (net 49 "/RX") (pintype "passive"))
-    (pad "R2" thru_hole oval (at -4.05 3.25 270) (size 0.75 1.8) (drill oval 0.45 1.5) (layers "*.Cu" "*.Mask")
-      (net 50 "/TX") (pintype "passive"))
-    (pad "S" thru_hole oval (at 4.05 2.4 270) (size 0.75 1.8) (drill oval 0.45 1.5) (layers "*.Cu" "*.Mask")
-      (net 26 "GND") (pintype "passive"))
-    (pad "T" thru_hole oval (at -4.05 11.4 270) (size 0.75 1.8) (drill oval 0.45 1.5) (layers "*.Cu" "*.Mask")
-      (net 4 "+5V") (pintype "passive"))
-    (pad "T" thru_hole oval (at 4.05 11.4 270) (size 0.75 1.8) (drill oval 0.45 1.5) (layers "*.Cu" "*.Mask")
-      (net 4 "+5V") (pintype "passive"))
-    (model "${KICAD_KBD_DIR}/kicad-packages3D/kbd.3dshapes/ST-0277D00-052-142.step"
-      (offset (xyz 0 -6.7 -2.1))
-      (scale (xyz 1 1 1))
-      (rotate (xyz 0 0 0))
-    )
-  )
   (footprint "Capacitor_SMD:C_0603_1608Metric" (layer "B.Cu")
     (at 99.185 102.2325 180)
@@
   )
   (footprint "Button_Switch_SMD:SW_SPST_SKQG_WithStem" (layer "B.Cu")
-    (at 89.83 74.0625 180)
+    (at 108.29 74.5425 180)
     (descr "ALPS 5.2mm Square Low-profile Type (Surface Mount) SKQG Series, With stem, http://www.alps.com/prod/info/E/HTML/Tact/SurfaceMount/SKQG/SKQGAFE010.html")
     (tags "SPST Button Switch")
@@
       (polygon
         (pts
-          (xy 88.83 72.7625)
-          (xy 85.83 72.7625)
-          (xy 85.83 75.3625)
-          (xy 88.83 75.3625)
+          (xy 107.29 73.2425)
+          (xy 104.29 73.2425)
+          (xy 104.29 75.8425)
+          (xy 107.29 75.8425)
         )
       )
@@
       (polygon
         (pts
-          (xy 93.83 72.7625)
-          (xy 90.83 72.7625)
-          (xy 90.83 75.3625)
-          (xy 93.83 75.3625)
+          (xy 112.29 73.2425)
+          (xy 109.29 73.2425)
+          (xy 109.29 75.8425)
+          (xy 112.29 75.8425)
         )
       )
@@
     (property "ki_keywords" "usb universal serial bus type-C USB2.0")
     (attr smd)
-    (fp_text reference "J1" (at 0 6.95) (layer "B.SilkS")
+    (fp_text reference "J1" (at 0 6.95 180) (layer "B.SilkS")
         (effects (font (size 1 1) (thickness 0.15)) (justify mirror))
     )
-    (fp_text value "TYPE-C-31-M-13C" (at 0 -3.4) (layer "B.Fab")
+    (fp_text value "TYPE-C-31-M-13C" (at 0 -3.4 180) (layer "B.Fab")
         (effects (font (size 1 1) (thickness 0.15)) (justify mirror))
     )
-    (fp_line (start -7 -2.1) (end -4.62 -2.1)
-      (stroke (width 0.1) (type default)) (layer "Edge.Cuts"))
     (fp_line (start -4.62 4.6) (end -4.62 -2.1)
-      (stroke (width 0.1) (type solid)) (layer "Edge.Cuts"))
-    (fp_line (start 4.62 -2.1) (end 7 -2.1)
-      (stroke (width 0.1) (type default)) (layer "Edge.Cuts"))
+      (stroke (width 0.1) (type solid)) (layer "B.CrtYd"))
+    (fp_line (start 4.62 -2.1) (end -4.62 -2.1)
+      (stroke (width 0.1) (type default)) (layer "B.CrtYd"))
     (fp_line (start 4.62 4.6) (end -4.62 4.6)
-      (stroke (width 0.1) (type default)) (layer "Edge.Cuts"))
+      (stroke (width 0.1) (type default)) (layer "B.CrtYd"))
     (fp_line (start 4.62 4.6) (end 4.62 -2.1)
-      (stroke (width 0.1) (type solid)) (layer "Edge.Cuts"))
+      (stroke (width 0.1) (type solid)) (layer "B.CrtYd"))
+    (fp_line (start -4.62 4.6) (end -4.62 -2.1)
+      (stroke (width 0.1) (type solid)) (layer "F.CrtYd"))
+    (fp_line (start 4.62 -2.1) (end -4.62 -2.1)
+      (stroke (width 0.1) (type default)) (layer "F.CrtYd"))
+    (fp_line (start 4.62 4.6) (end -4.62 4.6)
+      (stroke (width 0.1) (type default)) (layer "F.CrtYd"))
+    (fp_line (start 4.62 4.6) (end 4.62 -2.1)
+      (stroke (width 0.1) (type solid)) (layer "F.CrtYd"))
     (pad "A1" smd rect (at -3.25 5.35) (size 0.6 1.45) (layers "B.Cu" "B.Paste" "B.Mask")
       (net 26 "GND") (pinfunction "GND") (pintype "passive"))
@@
     )
   )
+  (footprint "kbd_local:ST-0277D00-052-142" (layer "B.Cu")
+    (at 166.68 94.2125 90)
+    (descr "USB Type-C receptacle for USB 2.0 and PD, http://www.krhro.com/uploads/soft/180320/1-1P320120243.pdf")
+    (tags "usb usb-c 2.0 pd")
+    (property "JLCPCB Part #" "C2837093")
+    (property "Sheetfile" "corne.kicad_sch")
+    (property "Sheetname" "")
+    (property "ki_description" "Audio Jack, 4 Poles (TRRS)")
+    (property "ki_keywords" "audio jack receptacle stereo headphones TRRS connector")
+    (attr smd)
+    (fp_text reference "J2" (at 0 -14.65 90) (layer "B.SilkS")
+        (effects (font (size 1 1) (thickness 0.15)) (justify mirror))
+    )
+    (fp_text value "ST-0277D00-052-142" (at 0 -16.2 90) (layer "B.Fab")
+        (effects (font (size 1 1) (thickness 0.15)) (justify mirror))
+    )
+    (fp_line (start -3.35 -13.5) (end 3.35 -13.5)
+      (stroke (width 0.1) (type solid)) (layer "B.CrtYd"))
+    (fp_line (start -3.35 0) (end -3.35 -13.5)
+      (stroke (width 0.1) (type solid)) (layer "B.CrtYd"))
+    (fp_line (start -3.35 0) (end 3.35 0)
+      (stroke (width 0.1) (type solid)) (layer "B.CrtYd"))
+    (fp_line (start 3.35 0) (end 3.35 -13.5)
+      (stroke (width 0.1) (type solid)) (layer "B.CrtYd"))
+    (fp_line (start -3.35 -13.5) (end 3.35 -13.5)
+      (stroke (width 0.1) (type solid)) (layer "F.CrtYd"))
+    (fp_line (start -3.35 0) (end -3.35 -13.5)
+      (stroke (width 0.1) (type solid)) (layer "F.CrtYd"))
+    (fp_line (start -3.35 0) (end 3.35 0)
+      (stroke (width 0.1) (type solid)) (layer "F.CrtYd"))
+    (fp_line (start 3.35 0) (end 3.35 -13.5)
+      (stroke (width 0.1) (type solid)) (layer "F.CrtYd"))
+    (pad "R1" thru_hole oval (at 4.05 -6 90) (size 0.75 1.8) (drill oval 0.45 1.5) (layers "*.Cu" "*.Mask")
+      (net 49 "/RX") (pintype "passive"))
+    (pad "R2" thru_hole oval (at -4.05 -3.25 90) (size 0.75 1.8) (drill oval 0.45 1.5) (layers "*.Cu" "*.Mask")
+      (net 50 "/TX") (pintype "passive"))
+    (pad "S" thru_hole oval (at 4.05 -2.4 90) (size 0.75 1.8) (drill oval 0.45 1.5) (layers "*.Cu" "*.Mask")
+      (net 26 "GND") (pintype "passive"))
+    (pad "T" thru_hole oval (at -4.05 -11.4 90) (size 0.75 1.8) (drill oval 0.45 1.5) (layers "*.Cu" "*.Mask")
+      (net 4 "+5V") (pintype "passive"))
+    (pad "T" thru_hole oval (at 4.05 -11.4 90) (size 0.75 1.8) (drill oval 0.45 1.5) (layers "*.Cu" "*.Mask")
+      (net 4 "+5V") (pintype "passive"))
+    (model "${KICAD_KBD_DIR}/kicad-packages3D/kbd.3dshapes/ST-0277D00-052-142.step"
+      (offset (xyz 0 -6.7 -2.1))
+      (scale (xyz 1 1 1))
+      (rotate (xyz 0 0 0))
+    )
+  )
   (footprint "Resistor_SMD:R_0603_1608Metric" (layer "B.Cu")
     (at 108.275 89.5625 180)
@@
   (gr_line (start 89.695 100.5375) (end 99.22 117.20625)
     (stroke (width 0.1) (type default)) (layer "F.Fab"))
+  (gr_text "Next: Change reset sqitch" (at 48.35 117.9625) (layer "Edge.Cuts")
+    (effects (font (size 2 2) (thickness 0.15)) (justify left bottom))
+  )
   (segment (start 161.4245 57.595625) (end 161.4245 56.877443) (width 0.25) (layer "B.Cu") (net 0))
   (segment (start 161.4245 76.645625) (end 161.4245 75.927443) (width 0.25) (layer "B.Cu") (net 0))

Commit message: Set each part
Parts:
- SMDSW1, SMDSW2: value SKQGADE010 -> TS-1088R-02026; footprint Button_Switch_SMD:SW_SPST_SKQG_WithStem -> kbd_local:TS-1088R-02026
- moved J5 80.2 mm to (100.2, 137.7), turned to 180 degrees
- moved J6 76.2 mm to (97.7, 137.7), turned to 180 degrees
- moved SMDSW2 47.0 mm to (68.6, 95.5)
- moved SMDSW1 46.5 mm to (68.6, 98.7)
- moved J4 43.1 mm to (105.2, 125.5), turned to 0 degrees
- moved C16 39.9 mm to (72.1, 88.6)
- moved R6 34.2 mm to (74.3, 93.7)
- moved R7 33.7 mm to (73.9, 91.1)
- moved U4 32.0 mm to (75.5, 97.4), turned to 0 degrees
- moved C10 16.4 mm to (98.5, 100.7)
- moved C2 16.3 mm to (99.2, 93.9), turned to -90 degrees
- moved C7 12.3 mm to (85.7, 99.3)
- moved ZD1 11.5 mm to (160.9, 51.0), turned to 0 degrees
- moved Y1 11.4 mm to (101.8, 95.9), turned to -90 degrees
- moved F1 10.4 mm to (150.2, 49.4), turned to -90 degrees
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Connections:
- D19 pad 1: unconnected-(D19-K-Pad1) -> /ROW0
- D19 pad 2: unconnected-(D19-A-Pad2) -> Net-(D19-A)
- D4 pad 2: unconnected-(D4-A-Pad2) -> Net-(D4-A)
- D6 pad 2: unconnected-(D6-A-Pad2) -> Net-(D6-A)
- EXD1 pad 2: unconnected-(EXD1-A-Pad2) -> Net-(EXD1-A)
- EXD2 pad 1: unconnected-(EXD2-K-Pad1) -> /ROW1
- EXD2 pad 2: unconnected-(EXD2-A-Pad2) -> Net-(EXD2-A)
- EXSW1 pad A: unconnected-(EXSW1-PadA) -> /RE0A
- EXSW1 pad B: unconnected-(EXSW1-PadB) -> /RE0B
- EXSW1 pad C: unconnected-(EXSW1-PadC) -> GND
- EXSW1 pad S1: unconnected-(EXSW1-PadS1) -> Net-(EXD1-A)
- EXSW1 pad S2: unconnected-(EXSW1-PadS2) -> /COL6
- EXSW2 pad S1: unconnected-(EXSW2-PadS1) -> Net-(EXD2-A)
- SW19 pad 2: unconnected-(SW19-Pad2) -> Net-(D19-A)
- SW4 pad 1: unconnected-(SW4-Pad1) -> /COL5
- SW4 pad 2: unconnected-(SW4-Pad2) -> Net-(D4-A)
- SW6 pad 1: unconnected-(SW6-Pad1) -> /COL4
- SW6 pad 2: unconnected-(SW6-Pad2) -> Net-(D6-A)
Routing:
- net (no net): track 22.0 -> 0.00 mm
- net Net-(EXD1-A): track 0.00 -> 6.79 mm
- net Net-(EXD2-A): track 0.00 -> 6.79 mm
- net unconnected-(EXSW1-PadS2): track 6.34 -> 0.00 mm
- net /COL6: track 6.34 -> 12.7 mm
- net Net-(D19-A): track 0.00 -> 2.83 mm
- net Net-(D4-A): track 0.00 -> 2.82 mm
- net Net-(D6-A): track 0.00 -> 2.82 mm
Other:
- board text added: "Next: Add lines"
- board text removed: "Next: Change reset sqitch"

Commit message: Add lines
Parts:
- removed J5, J6: Conn_01x06, Connector_PinHeader_2.54mm:PinHeader_1x06_P2.54mm_Vertical
- C1, C10, C11, C12, C13, C14, C15, C16, C2, C3, C4, C5, C6, C7, C8, C9: footprint Capacitor_SMD:C_0603_1608Metric -> Capacitor_SMD:C_0402_1005Metric
- moved R5 20.2 mm to (161.7, 64.8)
- moved R4 20.1 mm to (163.3, 64.8)
- moved C3 20.0 mm to (101.8, 98.2), turned to 0 degrees
- moved C16 19.0 mm to (87.3, 99.8), turned to 0 degrees
- moved J4 16.7 mm to (97.9, 110.6), turned to 180 degrees
- moved C7 16.2 mm to (101.8, 97.2), turned to 0 degrees
- moved ZD1 12.8 mm to (149.5, 45.1), turned to 90 degrees
- moved C13 11.5 mm to (92.3, 102.7), turned to -90 degrees
- moved U3 11.1 mm to (155.5, 55.3), turned to 90 degrees
- moved C14 9.60 mm to (90.9, 92.9)
- moved C15 8.82 mm to (89.7, 97.8)
- moved R7 8.29 mm to (77.1, 98.8)
- moved C4 7.74 mm to (89.7, 96.8)
- moved U4 7.39 mm to (82.8, 97.6)
- moved C6 6.22 mm to (145.0, 101.1), turned to 90 degrees
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Connections:
- U1 pad 34: /GPIO22 -> unconnected-(U1-GPIO22-Pad34)
- U1 pad 35: /GPIO23 -> unconnected-(U1-GPIO23-Pad35)
- U1 pad 36: /GPIO24 -> unconnected-(U1-GPIO24-Pad36)
- U1 pad 37: /GPIO25 -> unconnected-(U1-GPIO25-Pad37)
- U1 pad 38: /GPIO26 -> unconnected-(U1-GPIO26_ADC0-Pad38)
- U1 pad 39: /GPIO27 -> unconnected-(U1-GPIO27_ADC1-Pad39)
- U1 pad 40: /GPIO28 -> unconnected-(U1-GPIO28_ADC2-Pad40)
- U1 pad 41: /GPIO29 -> unconnected-(U1-GPIO29_ADC3-Pad41)
- U3 pad 1: /D- -> /D+
- U3 pad 10: /D- -> /D+
- U3 pad 5: /D+ -> /D-
- U3 pad 6: /D+ -> /D-
Routing:
- net GND: track 0.00 -> 645.6 mm, vias 0 -> 19
- net +5V: track 0.00 -> 528.8 mm, vias 0 -> 11
- net /ROW0: track 0.00 -> 195.6 mm, vias 0 -> 4
- net /ROW1: track 0.00 -> 182.9 mm, vias 0 -> 2
- net Net-(EXLED1-DIN): track 0.00 -> 170.2 mm
- net /COL5: track 0.00 -> 142.9 mm, vias 0 -> 9
- net /ROW2: track 0.00 -> 135.3 mm, vias 0 -> 2
- net /COL0: track 0.00 -> 113.8 mm, vias 0 -> 6
- net +3V3: track 0.00 -> 112.5 mm, vias 0 -> 10
- net /COL4: track 0.00 -> 111.8 mm, vias 0 -> 9
- net /RX: track 0.00 -> 105.4 mm, vias 0 -> 3
- net /COL6: track 12.7 -> 117.4 mm, vias 0 -> 4
- net /COL3: track 0.00 -> 100.9 mm, vias 0 -> 10
- net /RE0B: track 0.00 -> 100.2 mm, vias 0 -> 2
- net Net-(U1-USB_DP): track 0.00 -> 98.2 mm, vias 0 -> 4
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- added copper zone on B.Cu, net GND
Other:
- outline, holes or cut-outs redrawn
- board text added: "Edge of body"
- board text removed: "Next: Add lines"

Commit message: Update lines
Parts:
- C1, C2: value 20p -> 27p
- U4: footprint Package_SON:WSON-8-1EP_6x5mm_P1.27mm_EP3.4x4.3mm -> Package_SO:SOIC-8_5.23x5.23mm_P1.27mm
- Y1: value 12MHz 10pF -> 12MHz 18pF; footprint Crystal:Crystal_SMD_2520-4Pin_2.5x2.0mm -> Crystal:Crystal_SMD_3225-4Pin_3.2x2.5mm
Routing:
- net VBUS: track 19.8 -> 18.6 mm
- net Net-(J1-CC2): track 10.4 -> 9.79 mm
Other:
- outline, holes or cut-outs redrawn

Commit message: Update positions
Parts:
- moved R7 2.99 mm to (74.1, 98.9)
- moved R6 2.97 mm to (74.2, 97.0)
- moved SMDSW2 2.79 mm to (71.0, 97.5)
- moved SMDSW1 2.71 mm to (67.8, 97.5)
- moved U4 1.28 mm to (81.6, 97.5)
Routing:
- net /RX: track 105.4 -> 88.7 mm
- net /QSPI_SD1: track 18.1 -> 21.9 mm
- net /QSPI_SS: track 21.6 -> 25.2 mm
- net /QSPI_SD2: track 16.0 -> 19.4 mm
- net +3V3: track 112.5 -> 115.4 mm
- net Net-(U1-RUN): track 26.7 -> 29.5 mm
- net GND: track 646.1 -> 648.3 mm
- net +5V: track 528.8 -> 529.7 mm
- net /QSPI_SD0: track 7.45 -> 8.02 mm

Commit message: Fix some errors
Parts:
- moved C16 0.14 mm to (87.4, 100.0)
- moved C5 0.13 mm to (89.7, 98.9)
- moved C8 0.13 mm to (89.7, 100.0)
- moved C15 0.11 mm to (89.7, 97.9)
- moved C4 0.09 mm to (89.7, 96.9)
Routing:
- net GND: track 648.3 -> 650.3 mm

Commit message: Finish left hand
Routing:
- net GND: track 650.3 -> 650.9 mm
