File: pcb/corne.kicad_sch (KiCad schematic)
At the start: 107 parts, among them J1 TYPE-C-31-M-13C, J2 ST-0277D00-052-142, J3 Conn_01x04, J4 Conn_01x03, J5 Conn_01x06, J6 Conn_01x06, SW1 SW_Push, SW10 SW_Push, SW11 SW_Push, SW12 SW_Push, SW13 SW_Push, SW14 SW_Push, SW15 SW_Push, SW16 SW_Push, SW17 SW_Push, SW18 SW_Push, SW19 SW_Push, SW2 SW_Push, SW20 SW_Push, SW21 SW_Push, SW3 SW_Push, SW4 SW_Push, SW5 SW_Push, SW6 SW_Push, SW7 SW_Push, SW8 SW_Push, SW9 SW_Push, U1 RP2040, U2 NCP1117LPST33T3G, U3 TPD4E05U06DQAR, U4 W25Q128JVSIQ, Y1 12MHz 10pF

Commit message: Update pcb
Parts:
- SW1: footprint kbd:keyswitch_cherrymx_hotswap_1u -> kbd:keyswitch_cherrymx_hotswap_1.5u
Connections:
- net COL4: no longer SW6.1
- net COL5: no longer SW4.1
- net COL6: no longer EXSW1.S2
- net GND: no longer EXSW1.C
- net RE0A: no longer EXSW1.A
- net RE0B: no longer EXSW1.B
- net ROW0: no longer D19.1 (K)
- net ROW1: no longer EXD2.1 (K)
- net at D4.2 (A): no longer SW4.2
- net at D19.2 (A): no longer SW19.2
- net at D6.2 (A): no longer SW6.2
- net at EXSW1.S1: no longer EXD1.2 (A)
- net at EXD2.2 (A): no longer EXSW2.S1
Other:
- moved on the sheet: D19, EXD2, EXSW1, SW4, SW6
Changed lines of the file:
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@@
   (junction (at 195.58 224.79) (diameter 0) (color 0 0 0 0)
   )
-  (junction (at 231.14 120.65) (diameter 0) (color 0 0 0 0)
-  )
   (junction (at 27.94 185.42) (diameter 0) (color 0 0 0 0)
   )
@@
   (junction (at 215.9 143.51) (diameter 0) (color 0 0 0 0)
   )
-  (junction (at 243.84 105.41) (diameter 0) (color 0 0 0 0)
-  )
   (junction (at 241.3 143.51) (diameter 0) (color 0 0 0 0)
   )
@@
   (junction (at 76.2 111.76) (diameter 0) (color 0 0 0 0)
   )
-  (junction (at 190.5 113.03) (diameter 0) (color 0 0 0 0)
-  )
   (junction (at 109.22 99.06) (diameter 0) (color 0 0 0 0)
   )
@@
     (stroke (width 0) (type default))
   )
-  (wire (pts (xy 190.5 113.03) (xy 203.2 113.03))
-    (stroke (width 0) (type default))
-  )
   (wire (pts (xy 241.3 128.27) (xy 254 128.27))
     (stroke (width 0) (type default))
@@
     (stroke (width 0) (type default))
   )
-  (wire (pts (xy 231.14 105.41) (xy 231.14 120.65))
-    (stroke (width 0) (type default))
-  )
   (wire (pts (xy 63.5 30.48) (xy 69.85 30.48))
     (stroke (width 0) (type default))
@@
     (stroke (width 0) (type default))
   )
-  (wire (pts (xy 186.69 113.03) (xy 190.5 113.03))
+  (wire (pts (xy 186.69 113.03) (xy 203.2 113.03))
     (stroke (width 0) (type default))
   )
@@
     (stroke (width 0) (type default))
   )
-  (wire (pts (xy 231.14 120.65) (xy 231.14 135.89))
+  (wire (pts (xy 231.14 105.41) (xy 231.14 135.89))
     (stroke (width 0) (type default))
   )
@@
     (stroke (width 0) (type default))
   )
-  (wire (pts (xy 243.84 101.6) (xy 243.84 105.41))
-    (stroke (width 0) (type default))
-  )
   (wire (pts (xy 57.15 102.87) (xy 68.58 102.87))
     (stroke (width 0) (type default))
   )
-  (wire (pts (xy 243.84 105.41) (xy 243.84 120.65))
+  (wire (pts (xy 243.84 101.6) (xy 243.84 120.65))
     (stroke (width 0) (type default))
   )
@@
     )
   )
-  (symbol (lib_id "Device:D") (at 190.5 109.22 90) (unit 1)
+  (symbol (lib_id "Device:D") (at 200.66 81.28 90) (unit 1)
     (in_bom yes) (on_board yes) (dnp no)
-    (property "Reference" "D19" (at 187.96 109.22 0)
+    (property "Reference" "D19" (at 198.12 81.28 0)
       (effects (font (size 1.27 1.27)))
     )
-    (property "Value" "D" (at 193.04 109.22 0)
+    (property "Value" "D" (at 203.2 81.28 0)
       (effects (font (size 1.27 1.27)))
     )
-    (property "Footprint" "Diode_SMD:D_0603_1608Metric" (at 190.5 109.22 0)
+    (property "Footprint" "Diode_SMD:D_0603_1608Metric" (at 200.66 81.28 0)
       (effects (font (size 1.27 1.27)) hide)
     )
-    (property "Datasheet" "~" (at 190.5 109.22 0)
+    (property "Datasheet" "~" (at 200.66 81.28 0)
       (effects (font (size 1.27 1.27)) hide)
     )
-    (property "Sim.Device" "D" (at 190.5 109.22 0)
+    (property "Sim.Device" "D" (at 200.66 81.28 0)
       (effects (font (size 1.27 1.27)) hide)
     )
-    (property "Sim.Pins" "1=K 2=A" (at 190.5 109.22 0)
+    (property "Sim.Pins" "1=K 2=A" (at 200.66 81.28 0)
       (effects (font (size 1.27 1.27)) hide)
     )
@@
     )
   )
-  (symbol (lib_id "Device:RotaryEncoder_Switch") (at 274.32 102.87 180) (unit 1)
+  (symbol (lib_id "Device:RotaryEncoder_Switch") (at 278.13 106.68 180) (unit 1)
     (in_bom yes) (on_board yes) (dnp no)
-    (property "Reference" "EXSW1" (at 290.068 92.71 0)
+    (property "Reference" "EXSW1" (at 293.878 96.52 0)
       (effects (font (size 1.27 1.27)))
     )
-    (property "Value" "RotaryEncoder_Switch" (at 290.068 95.25 0)
+    (property "Value" "RotaryEncoder_Switch" (at 293.878 99.06 0)
       (effects (font (size 1.27 1.27)))
     )
-    (property "Footprint" "kbd_local:keyswitch_cherrymx_hotswap_1u_rotary_encoder_ec12" (at 278.13 106.934 0)
+    (property "Footprint" "kbd_local:keyswitch_cherrymx_hotswap_1u_rotary_encoder_ec12" (at 281.94 110.744 0)
       (effects (font (size 1.27 1.27)) hide)
     )
-    (property "Datasheet" "~" (at 274.32 109.474 0)
+    (property "Datasheet" "~" (at 278.13 113.284 0)
       (effects (font (size 1.27 1.27)) hide)
     )
@@
       (effects (font (size 1 1)))
     )
-    (property "Footprint" "kbd:keyswitch_cherrymx_hotswap_1u" (at 248.92 146.05 0)
+    (property "Footprint" "kbd:keyswitch_cherrymx_hotswap_1.5u" (at 248.92 146.05 0)
       (effects (font (size 1.27 1.27)) hide)
     )
@@
     )
   )
-  (symbol (lib_id "Device:D") (at 266.7 124.46 90) (unit 1)
+  (symbol (lib_id "Device:D") (at 303.53 237.49 90) (unit 1)
     (in_bom yes) (on_board yes) (dnp no)
-    (property "Reference" "EXD2" (at 264.16 124.46 0)
+    (property "Reference" "EXD2" (at 300.99 237.49 0)
       (effects (font (size 1.27 1.27)))
     )
-    (property "Value" "D" (at 269.24 124.46 0)
+    (property "Value" "D" (at 306.07 237.49 0)
       (effects (font (size 1.27 1.27)))
     )
-    (property "Footprint" "Diode_SMD:D_0603_1608Metric" (at 266.7 124.46 0)
+    (property "Footprint" "Diode_SMD:D_0603_1608Metric" (at 303.53 237.49 0)
       (effects (font (size 1.27 1.27)) hide)
     )
-    (property "Datasheet" "~" (at 266.7 124.46 0)
+    (property "Datasheet" "~" (at 303.53 237.49 0)
       (effects (font (size 1.27 1.27)) hide)
     )
-    (property "Sim.Device" "D" (at 266.7 124.46 0)
+    (property "Sim.Device" "D" (at 303.53 237.49 0)
       (effects (font (size 1.27 1.27)) hide)
     )
-    (property "Sim.Pins" "1=K 2=A" (at 266.7 124.46 0)
+    (property "Sim.Pins" "1=K 2=A" (at 303.53 237.49 0)
       (effects (font (size 1.27 1.27)) hide)
     )
@@
     )
   )
-  (symbol (lib_id "Switch:SW_Push") (at 236.22 120.65 0) (unit 1)
+  (symbol (lib_id "Switch:SW_Push") (at 201.93 39.37 0) (unit 1)
     (in_bom yes) (on_board yes) (dnp no)
-    (property "Reference" "SW6" (at 236.22 114.554 0)
+    (property "Reference" "SW6" (at 201.93 33.274 0)
       (effects (font (size 1 1)))
     )
-    (property "Value" "SW_Push" (at 236.22 116.586 0)
+    (property "Value" "SW_Push" (at 201.93 35.306 0)
       (effects (font (size 1 1)))
     )
-    (property "Footprint" "kbd:keyswitch_cherrymx_hotswap_1u" (at 236.22 115.57 0)
+    (property "Footprint" "kbd:keyswitch_cherrymx_hotswap_1u" (at 201.93 34.29 0)
       (effects (font (size 1.27 1.27)) hide)
     )
-    (property "Datasheet" "~" (at 236.22 115.57 0)
+    (property "Datasheet" "~" (at 201.93 34.29 0)
       (effects (font (size 1.27 1.27)) hide)
     )
@@
     )
   )
-  (symbol (lib_name "SW_Push_1") (lib_id "Switch:SW_Push") (at 248.92 105.41 0) (unit 1)
+  (symbol (lib_name "SW_Push_1") (lib_id "Switch:SW_Push") (at 248.92 76.2 0) (unit 1)
     (in_bom yes) (on_board yes) (dnp no)
-    (property "Reference" "SW4" (at 248.92 99.314 0)
+    (property "Reference" "SW4" (at 248.92 70.104 0)
       (effects (font (size 1 1)))
     )
-    (property "Value" "SW_Push" (at 248.92 101.346 0)
+    (property "Value" "SW_Push" (at 248.92 72.136 0)
       (effects (font (size 1 1)))
     )
-    (property "Footprint" "kbd:keyswitch_cherrymx_hotswap_1u" (at 248.92 100.33 0)
+    (property "Footprint" "kbd:keyswitch_cherrymx_hotswap_1u" (at 248.92 71.12 0)
       (effects (font (size 1.27 1.27)) hide)
     )
-    (property "Datasheet" "~" (at 248.92 100.33 0)
+    (property "Datasheet" "~" (at 248.92 71.12 0)
       (effects (font (size 1.27 1.27)) hide)
     )

Commit message: Set each part
Parts:
- SMDSW1, SMDSW2: value SKQGADE010 -> TS-1088R-02026; footprint Button_Switch_SMD:SW_SPST_SKQG_WithStem -> kbd_local:TS-1088R-02026; JLCPCB Part # C116647 -> C455280
Connections:
- net COL4: now also SW6.1
- net COL5: now also SW4.1
- net COL6: now also EXSW1.S2
- net GND: now also EXSW1.C
- net RE0A: now also EXSW1.A
- net RE0B: now also EXSW1.B
- net ROW0: now also D19.1 (K)
- net ROW1: now also EXD2.1 (K)
- net at D4.2 (A): now also SW4.2
- net at D19.2 (A): now also SW19.2
- net at D6.2 (A): now also SW6.2
- net at EXSW1.S1: now also EXD1.2 (A)
- net at EXD2.2 (A): now also EXSW2.S1
Other:
- moved on the sheet: D19, EXD2, EXSW1, SW4, SW6
Changed lines of the file:
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@@
   (junction (at 99.06 99.06) (diameter 0) (color 0 0 0 0)
   )
+  (junction (at 231.14 120.65) (diameter 0) (color 0 0 0 0)
+  )
   (junction (at 120.65 30.48) (diameter 0) (color 0 0 0 0)
   )
@@
   (junction (at 180.34 120.65) (diameter 0) (color 0 0 0 0)
   )
+  (junction (at 190.5 113.03) (diameter 0) (color 0 0 0 0)
+  )
   (junction (at 147.32 104.14) (diameter 0) (color 0 0 0 0)
   )
@@
   (junction (at 76.2 111.76) (diameter 0) (color 0 0 0 0)
   )
+  (junction (at 243.84 105.41) (diameter 0) (color 0 0 0 0)
+  )
   (junction (at 109.22 99.06) (diameter 0) (color 0 0 0 0)
   )
@@
     (stroke (width 0) (type default))
   )
+  (wire (pts (xy 190.5 113.03) (xy 203.2 113.03))
+    (stroke (width 0) (type default))
+  )
   (wire (pts (xy 91.44 99.06) (xy 91.44 107.95))
     (stroke (width 0) (type default))
@@
     (stroke (width 0) (type default))
   )
-  (wire (pts (xy 186.69 113.03) (xy 203.2 113.03))
+  (wire (pts (xy 186.69 113.03) (xy 190.5 113.03))
     (stroke (width 0) (type default))
   )
@@
     (stroke (width 0) (type default))
   )
+  (wire (pts (xy 243.84 105.41) (xy 243.84 120.65))
+    (stroke (width 0) (type default))
+  )
   (wire (pts (xy 241.3 205.74) (xy 241.3 224.79))
     (stroke (width 0) (type default))
@@
     (stroke (width 0) (type default))
   )
-  (wire (pts (xy 231.14 105.41) (xy 231.14 135.89))
+  (wire (pts (xy 231.14 105.41) (xy 231.14 120.65))
     (stroke (width 0) (type default))
   )
@@
     (stroke (width 0) (type default))
   )
+  (wire (pts (xy 231.14 120.65) (xy 231.14 135.89))
+    (stroke (width 0) (type default))
+  )
   (wire (pts (xy 27.94 185.42) (xy 40.64 185.42))
     (stroke (width 0) (type default))
@@
     (stroke (width 0) (type default))
   )
-  (wire (pts (xy 243.84 101.6) (xy 243.84 120.65))
+  (wire (pts (xy 243.84 101.6) (xy 243.84 105.41))
     (stroke (width 0) (type default))
   )
@@
     )
   )
-  (symbol (lib_id "Device:D") (at 200.66 81.28 90) (unit 1)
+  (symbol (lib_id "Device:D") (at 190.5 109.22 90) (unit 1)
     (in_bom yes) (on_board yes) (dnp no)
-    (property "Reference" "D19" (at 198.12 81.28 0)
+    (property "Reference" "D19" (at 187.96 109.22 0)
       (effects (font (size 1.27 1.27)))
     )
-    (property "Value" "D" (at 203.2 81.28 0)
+    (property "Value" "D" (at 193.04 109.22 0)
       (effects (font (size 1.27 1.27)))
     )
-    (property "Footprint" "Diode_SMD:D_0603_1608Metric" (at 200.66 81.28 0)
+    (property "Footprint" "Diode_SMD:D_0603_1608Metric" (at 190.5 109.22 0)
       (effects (font (size 1.27 1.27)) hide)
     )
-    (property "Datasheet" "~" (at 200.66 81.28 0)
+    (property "Datasheet" "~" (at 190.5 109.22 0)
       (effects (font (size 1.27 1.27)) hide)
     )
-    (property "Sim.Device" "D" (at 200.66 81.28 0)
+    (property "Sim.Device" "D" (at 190.5 109.22 0)
       (effects (font (size 1.27 1.27)) hide)
     )
-    (property "Sim.Pins" "1=K 2=A" (at 200.66 81.28 0)
+    (property "Sim.Pins" "1=K 2=A" (at 190.5 109.22 0)
       (effects (font (size 1.27 1.27)) hide)
     )
@@
     )
   )
-  (symbol (lib_id "Device:RotaryEncoder_Switch") (at 278.13 106.68 180) (unit 1)
+  (symbol (lib_id "Device:RotaryEncoder_Switch") (at 274.32 102.87 180) (unit 1)
     (in_bom yes) (on_board yes) (dnp no)
-    (property "Reference" "EXSW1" (at 293.878 96.52 0)
+    (property "Reference" "EXSW1" (at 290.068 92.71 0)
       (effects (font (size 1.27 1.27)))
     )
-    (property "Value" "RotaryEncoder_Switch" (at 293.878 99.06 0)
+    (property "Value" "RotaryEncoder_Switch" (at 290.068 95.25 0)
       (effects (font (size 1.27 1.27)))
     )
-    (property "Footprint" "kbd_local:keyswitch_cherrymx_hotswap_1u_rotary_encoder_ec12" (at 281.94 110.744 0)
+    (property "Footprint" "kbd_local:keyswitch_cherrymx_hotswap_1u_rotary_encoder_ec12" (at 278.13 106.934 0)
       (effects (font (size 1.27 1.27)) hide)
     )
-    (property "Datasheet" "~" (at 278.13 113.284 0)
+    (property "Datasheet" "~" (at 274.32 109.474 0)
       (effects (font (size 1.27 1.27)) hide)
     )
@@
     )
   )
-  (symbol (lib_id "Device:D") (at 303.53 237.49 90) (unit 1)
+  (symbol (lib_id "Device:D") (at 266.7 124.46 90) (unit 1)
     (in_bom yes) (on_board yes) (dnp no)
-    (property "Reference" "EXD2" (at 300.99 237.49 0)
+    (property "Reference" "EXD2" (at 264.16 124.46 0)
       (effects (font (size 1.27 1.27)))
     )
-    (property "Value" "D" (at 306.07 237.49 0)
+    (property "Value" "D" (at 269.24 124.46 0)
       (effects (font (size 1.27 1.27)))
     )
-    (property "Footprint" "Diode_SMD:D_0603_1608Metric" (at 303.53 237.49 0)
+    (property "Footprint" "Diode_SMD:D_0603_1608Metric" (at 266.7 124.46 0)
       (effects (font (size 1.27 1.27)) hide)
     )
-    (property "Datasheet" "~" (at 303.53 237.49 0)
+    (property "Datasheet" "~" (at 266.7 124.46 0)
       (effects (font (size 1.27 1.27)) hide)
     )
-    (property "Sim.Device" "D" (at 303.53 237.49 0)
+    (property "Sim.Device" "D" (at 266.7 124.46 0)
       (effects (font (size 1.27 1.27)) hide)
     )
-    (property "Sim.Pins" "1=K 2=A" (at 303.53 237.49 0)
+    (property "Sim.Pins" "1=K 2=A" (at 266.7 124.46 0)
       (effects (font (size 1.27 1.27)) hide)
     )
@@
       (effects (font (size 1.27 1.27)))
     )
-    (property "Value" "SKQGADE010" (at 50.8 120.142 0)
+    (property "Value" "TS-1088R-02026" (at 50.8 120.142 0)
       (effects (font (size 1.27 1.27)))
     )
-    (property "Footprint" "Button_Switch_SMD:SW_SPST_SKQG_WithStem" (at 50.8 120.65 0)
+    (property "Footprint" "kbd_local:TS-1088R-02026" (at 50.8 120.65 0)
       (effects (font (size 1.27 1.27)) hide)
     )
@@
       (effects (font (size 1.27 1.27)) hide)
     )
-    (property "JLCPCB Part #" "C116647" (at 50.8 125.73 0)
+    (property "JLCPCB Part #" "C455280" (at 50.8 125.73 0)
       (effects (font (size 1.27 1.27)) hide)
     )
@@
     )
   )
-  (symbol (lib_id "Switch:SW_Push") (at 201.93 39.37 0) (unit 1)
+  (symbol (lib_id "Switch:SW_Push") (at 236.22 120.65 0) (unit 1)
     (in_bom yes) (on_board yes) (dnp no)
-    (property "Reference" "SW6" (at 201.93 33.274 0)
+    (property "Reference" "SW6" (at 236.22 114.554 0)
       (effects (font (size 1 1)))
     )
-    (property "Value" "SW_Push" (at 201.93 35.306 0)
+    (property "Value" "SW_Push" (at 236.22 116.586 0)
       (effects (font (size 1 1)))
     )
-    (property "Footprint" "kbd:keyswitch_cherrymx_hotswap_1u" (at 201.93 34.29 0)
+    (property "Footprint" "kbd:keyswitch_cherrymx_hotswap_1u" (at 236.22 115.57 0)
       (effects (font (size 1.27 1.27)) hide)
     )
-    (property "Datasheet" "~" (at 201.93 34.29 0)
+    (property "Datasheet" "~" (at 236.22 115.57 0)
       (effects (font (size 1.27 1.27)) hide)
     )
@@
       (effects (font (size 1.27 1.27)))
     )
-    (property "Value" "SKQGADE010" (at 190.5 40.132 0)
+    (property "Value" "TS-1088R-02026" (at 190.5 40.132 0)
       (effects (font (size 1.27 1.27)))
     )
-    (property "Footprint" "Button_Switch_SMD:SW_SPST_SKQG_WithStem" (at 190.5 40.64 0)
+    (property "Footprint" "kbd_local:TS-1088R-02026" (at 190.5 40.64 0)
       (effects (font (size 1.27 1.27)) hide)
     )
@@
       (effects (font (size 1.27 1.27)) hide)
     )
-    (property "JLCPCB Part #" "C116647" (at 190.5 45.72 0)
+    (property "JLCPCB Part #" "C455280" (at 190.5 45.72 0)
       (effects (font (size 1.27 1.27)) hide)
     )
@@
     )
   )
-  (symbol (lib_name "SW_Push_1") (lib_id "Switch:SW_Push") (at 248.92 76.2 0) (unit 1)
+  (symbol (lib_name "SW_Push_1") (lib_id "Switch:SW_Push") (at 248.92 105.41 0) (unit 1)
     (in_bom yes) (on_board yes) (dnp no)
-    (property "Reference" "SW4" (at 248.92 70.104 0)
+    (property "Reference" "SW4" (at 248.92 99.314 0)
       (effects (font (size 1 1)))
     )
-    (property "Value" "SW_Push" (at 248.92 72.136 0)
+    (property "Value" "SW_Push" (at 248.92 101.346 0)
       (effects (font (size 1 1)))
     )
-    (property "Footprint" "kbd:keyswitch_cherrymx_hotswap_1u" (at 248.92 71.12 0)
+    (property "Footprint" "kbd:keyswitch_cherrymx_hotswap_1u" (at 248.92 100.33 0)
       (effects (font (size 1.27 1.27)) hide)
     )
-    (property "Datasheet" "~" (at 248.92 71.12 0)
+    (property "Datasheet" "~" (at 248.92 100.33 0)
       (effects (font (size 1.27 1.27)) hide)
     )

Commit message: Add lines
Parts:
- removed J5, J6: Conn_01x06, Connector_PinHeader_2.54mm:PinHeader_1x06_P2.54mm_Vertical, symbol Connector_Generic:Conn_01x06
- C1, C10, C11, C12, C13, C14, C15, C16, C2, C3, C4, C5, C6, C7, C8, C9: footprint Capacitor_SMD:C_0603_1608Metric -> Capacitor_SMD:C_0402_1005Metric
Connections:
- net D+: now also U3.1 (D1+), U3.10 (NC); no longer U3.5 (D2-), U3.6 (NC)
- net D-: now also U3.5 (D2-), U3.6 (NC); no longer U3.1 (D1+), U3.10 (NC)
- net GPIO22: no longer names the net of U1.34 (GPIO22)
- net GPIO23: no longer names the net of U1.35 (GPIO23)
- net GPIO24: no longer names the net of U1.36 (GPIO24)
- net GPIO25: no longer names the net of U1.37 (GPIO25)
- net GPIO26: no longer names the net of U1.38 (GPIO26_ADC0)
- net GPIO27: no longer names the net of U1.39 (GPIO27_ADC1)
- net GPIO28: no longer names the net of U1.40 (GPIO28_ADC2)
- net GPIO29: no longer names the net of U1.41 (GPIO29_ADC3)
- no-connect marks 4 -> 12
Other:
- note removed: "RP2040 original pins"

Commit message: Update lines
Parts:
- C1, C2: value 20p -> 27p
- U4: footprint Package_SON:WSON-8-1EP_6x5mm_P1.27mm_EP3.4x4.3mm -> Package_SO:SOIC-8_5.23x5.23mm_P1.27mm
- Y1: value 12MHz 10pF -> 12MHz 18pF; footprint Crystal:Crystal_SMD_2520-4Pin_2.5x2.0mm -> Crystal:Crystal_SMD_3225-4Pin_3.2x2.5mm; JLCPCB Part # C90603 -> C91749; MFR.Part # Q24FA20H0068700 -> Q22FA23V0041800
Changed lines of the file:
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@@
       (effects (font (size 1.27 1.27)))
     )
-    (property "Value" "12MHz 10pF" (at 52.07 177.8 90)
-      (effects (font (size 1.27 1.27)))
-    )
-    (property "Footprint" "Crystal:Crystal_SMD_2520-4Pin_2.5x2.0mm" (at 43.18 176.53 0)
+    (property "Value" "12MHz 18pF" (at 52.07 177.8 90)
+      (effects (font (size 1.27 1.27)))
+    )
+    (property "Footprint" "Crystal:Crystal_SMD_3225-4Pin_3.2x2.5mm" (at 43.18 176.53 0)
       (effects (font (size 1.27 1.27)) hide)
     )
@@
       (effects (font (size 1.27 1.27)) hide)
     )
-    (property "Description" "12MHz 10pF ±10ppm SMD2520-4P Crystals ROHS" (at 43.18 176.53 90)
-      (effects (font (size 1.27 1.27)) hide)
-    )
-    (property "MFR.Part #" "Q24FA20H0068700" (at 43.18 176.53 90)
-      (effects (font (size 1.27 1.27)) hide)
-    )
-    (property "JLCPCB Part #" "C90603" (at 43.18 176.53 90)
+    (property "Description" "12MHz 18pF ±20ppm SMD3225-4P Crystals ROHS" (at 43.18 176.53 90)
+      (effects (font (size 1.27 1.27)) hide)
+    )
+    (property "MFR.Part #" "Q22FA23V0041800" (at 43.18 176.53 90)
+      (effects (font (size 1.27 1.27)) hide)
+    )
+    (property "JLCPCB Part #" "C91749" (at 43.18 176.53 90)
       (effects (font (size 1.27 1.27)) hide)
     )
@@
       (effects (font (size 1.27 1.27)) (justify left))
     )
-    (property "Footprint" "Package_SON:WSON-8-1EP_6x5mm_P1.27mm_EP3.4x4.3mm" (at 228.6 53.34 0)
+    (property "Footprint" "Package_SO:SOIC-8_5.23x5.23mm_P1.27mm" (at 228.6 53.34 0)
       (effects (font (size 1.27 1.27)) hide)
     )
@@
       (effects (font (size 1.27 1.27)) (justify left))
     )
-    (property "Value" "20p" (at 34.29 172.72 90)
+    (property "Value" "27p" (at 34.29 172.72 90)
       (effects (font (size 1.27 1.27)) (justify left))
     )
@@
       (effects (font (size 1.27 1.27)) (justify left))
     )
-    (property "Value" "20p" (at 34.29 182.88 90)
-      (effects (font (size 1.27 1.27)) (justify left))
-    )
+    (property "Value" "27p" (at 34.29 182.88 90)
+      (effects (font (size 1.27 1.27)) (justify left))
+    )
