File: pcb/corne.kicad_sch (KiCad schematic)
At the start: 105 parts, among them J1 TYPE-C-31-M-13C, J2 ST-0277D00-052-142, J3 Conn_01x04, J4 Conn_01x03, SW1 SW_Push, SW10 SW_Push, SW11 SW_Push, SW12 SW_Push, SW13 SW_Push, SW14 SW_Push, SW15 SW_Push, SW16 SW_Push, SW17 SW_Push, SW18 SW_Push, SW19 SW_Push, SW2 SW_Push, SW20 SW_Push, SW21 SW_Push, SW3 SW_Push, SW4 SW_Push, SW5 SW_Push, SW6 SW_Push, SW7 SW_Push, SW8 SW_Push, SW9 SW_Push, U1 RP2040, U2 NCP1117LPST33T3G, U3 TPD4E05U06DQAR, U4 W25Q128JVSIQ, Y1 12MHz 18pF

Commit message: Update pcb
Parts:
- removed C1, C2: 27p, Capacitor_SMD:C_0402_1005Metric, symbol Device:C_Small
- removed C10, C12, C13, C14, C15, C3, C4, C7, C9: 100n, Capacitor_SMD:C_0402_1005Metric, symbol Device:C_Small
- removed C11, C6: 10u, Capacitor_SMD:C_0402_1005Metric, symbol Device:C_Small
- removed C16, C5, C8: 1u, Capacitor_SMD:C_0402_1005Metric, symbol Device:C_Small
- removed D1, D10, D11, D12, D13, D14, D15, D16, D17, D18, D19, D2, D20, D21, D3, D4, D5, D6, D7, D8, D9, EXD1, EXD2: D, Diode_SMD:D_0603_1608Metric, symbol Device:D
- removed EXLED1, EXLED2, LED1, LED10, LED11, LED12, LED13, LED14, LED15, LED16, LED17, LED18, LED19, LED2, LED20, LED21, LED3, LED4, LED5, LED6, LED7, LED8, LED9: YS-SK6812MINI-E, kbd_local:YS-SK6812MINI-E, symbol kbd_local:YS-SK6812MINI-E
- removed EXSW1, EXSW2: RotaryEncoder_Switch, kbd_local:keyswitch_cherrymx_hotswap_1u_rotary_encoder_ec12, symbol Device:RotaryEncoder_Switch
- removed F1: BSMD0603-050-12V, Fuse:Fuse_0603_1608Metric, symbol Device:Fuse
- removed J1: TYPE-C-31-M-13C, kbd_local:TYPE-C-31-M-13C, symbol Connector:USB_C_Receptacle_USB2.0
- removed J2: ST-0277D00-052-142, kbd_local:ST-0277D00-052-142, symbol Connector_Audio:AudioJack4
- removed J3: Conn_01x04, kbd_local:OLED, symbol Connector_Generic:Conn_01x04
- removed J4: Conn_01x03, Connector_PinHeader_2.54mm:PinHeader_1x03_P2.54mm_Vertical, symbol Connector_Generic:Conn_01x03
- removed R1, R2: 5.1k, Resistor_SMD:R_0603_1608Metric, symbol Device:R_Small
- removed R3, R6: 1k, Resistor_SMD:R_0603_1608Metric, symbol Device:R
- removed R4, R5: 27, Resistor_SMD:R_0603_1608Metric, symbol Device:R_Small
- removed R7: 10k, Resistor_SMD:R_0603_1608Metric, symbol Device:R
- removed SMDSW1, SMDSW2: TS-1088R-02026, kbd_local:TS-1088R-02026, symbol Switch:SW_Push
- removed SW1: SW_Push, kbd:keyswitch_cherrymx_hotswap_1.5u, symbol Switch:SW_Push
- removed SW10, SW11, SW12, SW13, SW14, SW15, SW16, SW17, SW18, SW19, SW2, SW20, SW21, SW3, SW4, SW5, SW6, SW7, SW8, SW9: SW_Push, kbd:keyswitch_cherrymx_hotswap_1u, symbol Switch:SW_Push
- removed U1: RP2040, Package_DFN_QFN:QFN-56-1EP_7x7mm_P0.4mm_EP3.2x3.2mm, symbol MCU_RaspberryPi:RP2040
- removed U2: NCP1117LPST33T3G, Package_TO_SOT_SMD:SOT-223-3_TabPin2, symbol Regulator_Linear:NCP1117-3.3_SOT223
- removed U3: TPD4E05U06DQAR, Package_SON:USON-10_2.5x1.0mm_P0.5mm, symbol Power_Protection:TPD4EUSB30
- removed U4: W25Q128JVSIQ, Package_SO:SOIC-8_5.23x5.23mm_P1.27mm, symbol Memory_Flash:W25Q128JVS
- removed Y1: 12MHz 18pF, Crystal:Crystal_SMD_3225-4Pin_3.2x2.5mm, symbol Device:Crystal_GND24_Small
- removed ZD1: ESD5Z5V0C, Diode_SMD:D_SOD-523, symbol Diode:ESD5Zxx
Connections:
- no-connect marks 12 -> 0
Other:
- added sheet left (left.kicad_sch)
- added sheet right (right.kicad_sch)
- note removed: "DEBUG"
- note removed: "Extention"
- note removed: "Flash memory"
- note removed: "Key switches"
- note removed: "LDO"
- note removed: "LEDs"
- note removed: "MCU RP2040"
- note removed: "OLED"
- note removed: "POWER"
- note removed: "SPLIT_HAND_PIN"
- note removed: "T(4,5), R1(3), R2(2), S(1)"
- note removed: "TRRS"
- note removed: "USB ESD"
- note removed: "VBUS ESD"
- note removed: "boot switch"
- note removed: "close to pin 44"
- note removed: "close to pin 45"
- note removed: "left R1:RX, R2:TX right R1:TX, R2:RX"
