File: pcb/common/right.kicad_sch (KiCad schematic)
At the start: 87 parts

Commit message: Update footprints and sch
Parts:
- added rJP1: SolderJumper_2_Bridged, Jumper:SolderJumper-2_P1.3mm_Open_RoundedPad1.0x1.5mm, symbol Jumper:SolderJumper_2_Bridged
Connections:
- net KEY1: now also rU?.30 (GPIO19); no longer rU?.29 (GPIO18)
- net KEY12: now also rU?.4 (GPIO2); no longer rU?.6 (GPIO4)
- net KEY13: now also rU?.5 (GPIO3); no longer rU?.7 (GPIO5)
- net KEY14: now also rU?.6 (GPIO4); no longer rU?.8 (GPIO6)
- net KEY15: now also rU?.7 (GPIO5); no longer rU?.9 (GPIO7)
- net KEY16: now also rU?.29 (GPIO18); no longer rU?.14 (GPIO11)
- net KEY17: now also rU?.17 (GPIO14); no longer rU?.12 (GPIO9)
- net KEY18: now also rU?.12 (GPIO9); no longer rU?.18 (GPIO15)
- net KEY19: now also rU?.11 (GPIO8); no longer rU?.17 (GPIO14)
- net KEY2: now also rU?.34 (GPIO22); no longer rU?.36 (GPIO24)
- net KEY20: now also rU?.14 (GPIO11); no longer rU?.11 (GPIO8)
- net KEY21: now also rU?.18 (GPIO15); no longer rU?.13 (GPIO10)
- net KEY3: now also rU?.38 (GPIO26_ADC0); no longer rU?.40 (GPIO28_ADC2)
- net KEY4: now also rU?.39 (GPIO27_ADC1); no longer rU?.4 (GPIO2)
- net KEY5: now also rU?.3 (GPIO1); no longer rU?.5 (GPIO3)
- net KEY6: now also rU?.40 (GPIO28_ADC2); no longer rU?.3 (GPIO1)
- net KEYEX1: now also rU?.37 (GPIO25); no longer rU?.39 (GPIO27_ADC1)
- net KEYEX2: now also rU?.35 (GPIO23); no longer rU?.37 (GPIO25)
- net LED: now also rU?.13 (GPIO10); no longer rU?.30 (GPIO19)
- net RE0A: now also rU?.36 (GPIO24); no longer rU?.38 (GPIO26_ADC0)
- net RE1A: now also rU?.8 (GPIO6); no longer rU?.34 (GPIO22)
- net REB: now also rU?.9 (GPIO7); no longer rU?.35 (GPIO23)
- net at rLED?.2 (DOUT), rLED?.4 (DIN): now also rJP1.1 (A)
- net at rEXLED?.4 (DIN), rLED?.2 (DOUT): now also rJP1.2 (B)
Other:
- moved on the sheet: rD?
