File: plates/3x5/pcb/plate-top-alps-ex.kicad_pcb (KiCad board)
At the start: 2 copper layers, 135.1 x 94.4 mm, 0 parts

Commit message: Update pcb plate files
Other:
- board size 135.1 x 94.4 mm -> 116.1 x 94.4 mm
