File: plates/3x5/pcb/plate-top-cherrymx-ex.kicad_pcb (KiCad board)
At the start: 2 copper layers, 116.1 x 94.4 mm, 0 parts

Commit message: Update pcb plate files
Other:
- outline, holes or cut-outs redrawn
