File: plates/3x6/pcb/plate-top-alps-ex.kicad_pcb (KiCad board)
At the start: 2 copper layers, 135.1 x 94.4 mm, 0 parts

Commit message: Update pcb plate files
Other:
- outline, holes or cut-outs redrawn
Changed lines of the file:
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@@
   (gr_arc (start -83.637454 1.142234) (mid -83.283901 1.288681) (end -83.137454 1.642234)
     (stroke (width 0.2) (type solid)) (layer "Edge.Cuts"))
+  (gr_arc (start -22.437454 13.548484) (mid -22.291007 13.194931) (end -21.937454 13.048484)
+    (stroke (width 0.2) (type solid)) (layer "Edge.Cuts"))
   (gr_curve (pts (xy -23.937766 -19.506396) (xy -23.831657 -19.473167) (xy -23.735679 -19.419979) (xy -23.647391 -19.346015))
     (stroke (width 0.2) (type solid)) (layer "Edge.Cuts"))
@@
   (gr_arc (start -64.587454 17.810984) (mid -64.233901 17.957431) (end -64.087454 18.310984)
     (stroke (width 0.2) (type solid)) (layer "Edge.Cuts"))
+  (gr_arc (start -21.937454 25.848484) (mid -22.291007 25.702037) (end -22.437454 25.348484)
+    (stroke (width 0.2) (type solid)) (layer "Edge.Cuts"))
   (gr_arc (start -70.062515 42.123363) (mid -69.916068 41.76981) (end -69.562515 41.623363)
     (stroke (width 0.2) (type solid)) (layer "Edge.Cuts"))
@@
     (stroke (width 0.2) (type solid)) (layer "Edge.Cuts"))
   (gr_line (start -45.053346 -17.409461) (end -45.053346 -5.609461)
+    (stroke (width 0.2) (type solid)) (layer "Edge.Cuts"))
+  (gr_line (start -22.437454 13.548484) (end -22.437454 25.348484)
     (stroke (width 0.2) (type solid)) (layer "Edge.Cuts"))
   (gr_line (start -34.384336 62.369967) (end -17.186286 69.984068)
@@
   (gr_line (start -117.687457 37.254739) (end -117.687457 25.454739)
     (stroke (width 0.2) (type solid)) (layer "Edge.Cuts"))
+  (gr_line (start -21.937454 25.848484) (end -7.437454 25.848484)
+    (stroke (width 0.2) (type solid)) (layer "Edge.Cuts"))
   (gr_line (start -98.153346 -5.108004) (end -83.653346 -5.108004)
     (stroke (width 0.2) (type solid)) (layer "Edge.Cuts"))
@@
   (gr_curve (pts (xy -138.935579 -17.072115) (xy -138.842516 -17.120446) (xy -138.754364 -17.143845) (xy -138.677381 -17.155925))
     (stroke (width 0.2) (type solid)) (layer "Edge.Cuts"))
+  (gr_arc (start -6.937454 25.348484) (mid -7.083901 25.702037) (end -7.437454 25.848484)
+    (stroke (width 0.2) (type solid)) (layer "Edge.Cuts"))
   (gr_curve (pts (xy -4.262502 43.051692) (xy -4.262502 43.114725) (xy -4.262502 43.181926) (xy -4.278945 43.259681))
     (stroke (width 0.2) (type solid)) (layer "Edge.Cuts"))
@@
     (stroke (width 0.2) (type solid)) (layer "Edge.Cuts"))
   (gr_arc (start -45.537515 20.192232) (mid -45.183962 20.338679) (end -45.037515 20.692232)
+    (stroke (width 0.2) (type solid)) (layer "Edge.Cuts"))
+  (gr_line (start -22.437454 -5.501516) (end -22.437454 6.298484)
+    (stroke (width 0.2) (type solid)) (layer "Edge.Cuts"))
+  (gr_arc (start -21.937454 6.798484) (mid -22.291007 6.652037) (end -22.437454 6.298484)
     (stroke (width 0.2) (type solid)) (layer "Edge.Cuts"))
   (gr_curve (pts (xy -4.278945 43.259681) (xy -4.295387 43.337436) (xy -4.322593 43.398884) (xy -4.34811 43.456521))
@@
   (gr_arc (start -83.153346 -5.608004) (mid -83.299793 -5.254451) (end -83.653346 -5.108004)
     (stroke (width 0.2) (type solid)) (layer "Edge.Cuts"))
+  (gr_arc (start -22.437454 -5.501516) (mid -22.291007 -5.855069) (end -21.937454 -6.001516)
+    (stroke (width 0.2) (type solid)) (layer "Edge.Cuts"))
   (gr_line (start -64.587454 30.610984) (end -79.087454 30.610984)
     (stroke (width 0.2) (type solid)) (layer "Edge.Cuts"))
@@
   (gr_arc (start -121.737454 5.904733) (mid -121.383901 6.05118) (end -121.237454 6.404733)
     (stroke (width 0.2) (type solid)) (layer "Edge.Cuts"))
+  (gr_line (start -6.937454 25.348484) (end -6.937454 13.548484)
+    (stroke (width 0.2) (type solid)) (layer "Edge.Cuts"))
   (gr_curve (pts (xy -82.234742 -23.704855) (xy -82.201513 -23.810964) (xy -82.148325 -23.906942) (xy -82.074361 -23.99523))
     (stroke (width 0.2) (type solid)) (layer "Edge.Cuts"))
   (gr_arc (start -102.687457 24.954739) (mid -102.333903 25.101185) (end -102.187457 25.454739)
     (stroke (width 0.2) (type solid)) (layer "Edge.Cuts"))
+  (gr_line (start -7.437454 -6.001516) (end -21.937454 -6.001516)
+    (stroke (width 0.2) (type solid)) (layer "Edge.Cuts"))
   (gr_curve (pts (xy -138.803036 41.736134) (xy -138.909145 41.702905) (xy -139.005123 41.649717) (xy -139.093411 41.575753))
     (stroke (width 0.2) (type solid)) (layer "Edge.Cuts"))
@@
   (gr_line (start -117.203346 -0.345661) (end -102.703346 -0.345661)
     (stroke (width 0.2) (type solid)) (layer "Edge.Cuts"))
+  (gr_line (start -21.937454 6.798484) (end -7.437454 6.798484)
+    (stroke (width 0.2) (type solid)) (layer "Edge.Cuts"))
   (gr_arc (start -121.737456 24.954736) (mid -121.383903 25.101183) (end -121.237456 25.454736)
+    (stroke (width 0.2) (type solid)) (layer "Edge.Cuts"))
+  (gr_arc (start -6.937454 6.298484) (mid -7.083901 6.652037) (end -7.437454 6.798484)
     (stroke (width 0.2) (type solid)) (layer "Edge.Cuts"))
   (gr_arc (start -83.137454 13.442234) (mid -83.283901 13.795787) (end -83.637454 13.942234)
@@
   (gr_line (start -64.103346 -7.989276) (end -64.103346 -19.789276)
     (stroke (width 0.2) (type solid)) (layer "Edge.Cuts"))
+  (gr_line (start -6.937454 6.298484) (end -6.937454 -5.501516)
+    (stroke (width 0.2) (type solid)) (layer "Edge.Cuts"))
   (gr_line (start -136.237456 24.954736) (end -121.737456 24.954736)
     (stroke (width 0.2) (type solid)) (layer "Edge.Cuts"))
@@
   (gr_line (start -81.884744 41.779734) (end -72.644369 57.950377)
     (stroke (width 0.2) (type solid)) (layer "Edge.Cuts"))
+  (gr_arc (start -7.437454 13.048484) (mid -7.083901 13.194931) (end -6.937454 13.548484)
+    (stroke (width 0.2) (type solid)) (layer "Edge.Cuts"))
   (gr_line (start -70.062515 53.923363) (end -70.062515 42.123363)
     (stroke (width 0.2) (type solid)) (layer "Edge.Cuts"))
@@
   (gr_curve (pts (xy -139.208478 -16.85137) (xy -139.140428 -16.932599) (xy -139.048782 -17.013323) (xy -138.935579 -17.072115))
     (stroke (width 0.2) (type solid)) (layer "Edge.Cuts"))
+  (gr_arc (start -7.437454 -6.001516) (mid -7.083901 -5.855069) (end -6.937454 -5.501516)
+    (stroke (width 0.2) (type solid)) (layer "Edge.Cuts"))
   (gr_line (start -136.237454 18.704733) (end -121.737454 18.704733)
     (stroke (width 0.2) (type solid)) (layer "Edge.Cuts"))
@@
   (gr_curve (pts (xy -4.276992 -16.433665) (xy -4.262502 -16.341329) (xy -4.262502 -16.253574) (xy -4.262502 -16.16875))
     (stroke (width 0.2) (type solid)) (layer "Edge.Cuts"))
+  (gr_line (start -7.437454 13.048484) (end -21.937454 13.048484)
+    (stroke (width 0.2) (type solid)) (layer "Edge.Cuts"))
   (gr_arc (start -79.087454 30.610984) (mid -79.441007 30.464537) (end -79.587454 30.110984)
