File: plates/3x6/pcb/plate-top-cherrymx-ex.kicad_pcb (KiCad board)
At the start: 2 copper layers, 116.1 x 94.4 mm, 0 parts

Commit message: Update pcb plate files
Other:
- board size 116.1 x 94.4 mm -> 135.1 x 94.4 mm
