File: plates/3x6/pcb/plate-top-cherrymx.kicad_pcb (KiCad board)
At the start: 2 copper layers, 135.1 x 94.4 mm, 0 parts

Commit message: Update pcb plate files
Other:
- outline, holes or cut-outs redrawn
